File: hardware/led.kicad_sch (KiCad schematic)
At the start: 0 parts

Commit message: wip: schematic sheets in progress (led)
Co-Authored-By: Claude Opus 5.5 <noreply@anthropic.com>
Claude-Session: https://claude.ai/code/session_01RFaS5jnC9tnPam9GBgmGnG
Parts:
- added D5: green, lib:LED_0402_1005Metric, symbol Device:LED
- added D6: blue, lib:LED_0402_1005Metric, symbol Device:LED
- added R85, R86: 150R, lib:R_0201_0603Metric_W, symbol Device:R
Connections:
- new net: D6.1 (K), R86.1
- new net: D5.1 (K), R85.1
- new net +3V3: D5.2 (A), D6.2 (A)
- new net LED0: R85.2
- new net LED1: R86.2
Other:
- note added: "status LEDs"
