File: hardware/led.kicad_sch (KiCad schematic)
At the start: 4 parts

Commit message: wip: schematic integration in progress (saved after container restart)
Co-Authored-By: Claude Opus 5.5 <noreply@anthropic.com>
Claude-Session: https://claude.ai/code/session_01RFaS5jnC9tnPam9GBgmGnG
Connections:
- net D6_K: now reaches D6.1 (K), R86.1
- net D5_K: now reaches D5.1 (K), R85.1
Changed lines of the file:
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@@
+	(wire
+		(pts
+			(xy 66.04 64.77) (xy 66.04 71.12)
+		)
+		(stroke
+			(width 0)
+			(type default)
+		)
+	)
+	(wire
+		(pts
+			(xy 45.72 64.77) (xy 45.72 71.12)
+		)
+		(stroke
+			(width 0)
+			(type default)
+		)
+	)
+	(wire
+		(pts
+			(xy 66.04 40.64) (xy 66.04 45.72)
+		)
+		(stroke
+			(width 0)
+			(type default)
+		)
+	)
+	(wire
+		(pts
+			(xy 45.72 40.64) (xy 45.72 45.72)
+		)
+		(stroke
+			(width 0)
+			(type default)
+		)
+	)
 	(wire
 		(pts
@@
 	(wire
 		(pts
-			(xy 66.04 40.64) (xy 66.04 45.72)
+			(xy 45.72 53.34) (xy 45.72 57.15)
 		)
 		(stroke
@@
 		)
 	)
-	(wire
-		(pts
-			(xy 45.72 40.64) (xy 45.72 45.72)
-		)
-		(stroke
-			(width 0)
-			(type default)
-		)
-	)
-	(wire
-		(pts
-			(xy 66.04 64.77) (xy 66.04 71.12)
-		)
-		(stroke
-			(width 0)
-			(type default)
-		)
-	)
-	(wire
-		(pts
-			(xy 45.72 64.77) (xy 45.72 71.12)
-		)
-		(stroke
-			(width 0)
-			(type default)
-		)
-	)
-	(wire
-		(pts
-			(xy 45.72 53.34) (xy 45.72 57.15)
-		)
-		(stroke
-			(width 0)
-			(type default)
+	(label "D5_K"
+		(at 45.72 55.88 180)
+		(effects
+			(font
+				(size 1.27 1.27)
+			)
+			(justify right bottom)
+		)
+	)
+	(label "D6_K"
+		(at 66.04 55.88 180)
+		(effects
+			(font
+				(size 1.27 1.27)
+			)
+			(justify right bottom)
+		)
+	)
+	(hierarchical_label "LED1"
+		(shape input)
+		(at 66.04 71.12 270)
+		(effects
+			(font
+				(size 1.27 1.27)
+			)
+			(justify right)
 		)
 	)
@@
 		(shape input)
 		(at 45.72 71.12 270)
-		(effects
-			(font
-				(size 1.27 1.27)
-			)
-			(justify right)
-		)
-	)
-	(hierarchical_label "LED1"
-		(shape input)
-		(at 66.04 71.12 270)
 		(effects
 			(font
@@
 		(in_pos_files no)
 		(dnp no)
-		(property "Reference" "#PWR01"
+		(property "Reference" "#PWR230"
 			(at 45.72 44.45 0)
 			(hide yes)
@@
 			(project "OpenAIO-Whoop"
 				(path "/2c3a7206-1e66-4d43-a02f-491225e20dd6/0a9dca22-7345-53f8-9367-07faa3e8899c"
-					(reference "#PWR01")
+					(reference "#PWR230")
 					(unit 1)
 				)
@@
 		(in_pos_files no)
 		(dnp no)
-		(property "Reference" "#PWR02"
+		(property "Reference" "#PWR231"
 			(at 66.04 44.45 0)
 			(hide yes)
@@
 			(project "OpenAIO-Whoop"
 				(path "/2c3a7206-1e66-4d43-a02f-491225e20dd6/0a9dca22-7345-53f8-9367-07faa3e8899c"
-					(reference "#PWR02")
+					(reference "#PWR231")
 					(unit 1)
 				)

Commit message: WIP final schematic (D111/D113): GPIO map, D100 oscillator, final footprints, lineup power-net names; mid-run snapshot, not yet verified (ERC/netlist/DRU regen pending)
Co-Authored-By: Claude Opus 5.5 <noreply@anthropic.com>
Claude-Session: https://claude.ai/code/session_01RFaS5jnC9tnPam9GBgmGnG
Parts:
- D5, D6: footprint lib:LED_0402_1005Metric -> lib:LED_0402_1005Metric_L
- R85, R86: footprint lib:R_0201_0603Metric_W -> lib:R_0201_0603Metric_L
Connections:
- net +3V3 renamed +3.3V
Changed lines of the file:
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@@
 		)
 	)
-	(text_box "STATUS LEDS (D5 D6 R85 R86)  source: OpenFC-Lite-Mini hardware/rp2350a.kicad_sch 'status LED' block (R52 + R53 2x 75R, D2 XL-1005UBC), copied and adapted: sink drive per hardware/sch_contract.json and research/PINMAP.md, 2x 75R -> one 150R 0201, second column for LED1.\nCircuit: +3V3 -> LED -> 150R -> GPIO, the pin sinks (contract). Betaflight default polarity, low = on, no LEDx_INVERTED: LED0_PIN PA7 (GPIO7, green D5), LED1_PIN PA26 (GPIO26, blue D6).\nDatasheet check (XINGLIGHT XL-1005UGC / UBC, 0402): VF 2.7-3.3 / 2.6-3.4 V at 20 mA, IF max 20 mA, PD 70 mW, VR 5 V. At a few mA the InGaN VF is about 0.2-0.3 V lower (inferred), so with VOL <= 0.5 V at 4 mA drive (RP2350 DS) the LED current is about 0.5-5 mA, typ. 2-3 mA, hard ceiling (3.3 - 2.4) / 150R = 6 mA: LED, 0201 resistor (<= 5.4 mW of 50 mW) and GPIO (4 mA setting, 100 mA IOVSS sum) all inside their ratings; brightness at 1-3 mA is about 17-135 mcd green and 4-36 mcd blue (Iv scaled from 350-900 / 80-240 mcd at 20 mA), enough for an indicator. Reverse bias is 0 V when the pin drives high (IOVDD = +3V3).\nReset state: RP2350 pads come up with the pull-down on (PDE = 1, 36-113 kOhm), so both LEDs may glow faintly (about 10-30 uA) until Betaflight drives the pins and in BOOTSEL mode. Accepted, cosmetic.\nPlacement (P5): bottom side, fc_core region (bom_plan); the R may sit at either end of the LED, slow signal (D33). Pins LED0/LED1 = root nets /LED0, /LED1 (RP2350A).\nP4 closed here: bom_plan R85/R86 'P4 checks brightness vs Vf' (above). P4-14 fields: RC0201FR-07150RL is a stocked Yageo RC_L part (Element14 4008725, RS 198-7568: 150R 1 % 50 mW 25 V); no LCSC number known, field left empty (contract open item A9-LCSC)."
+	(text_box "STATUS LEDS (D5 D6 R85 R86)  source: OpenFC-Lite-Mini hardware/rp2350a.kicad_sch 'status LED' block (R52 + R53 2x 75R, D2 XL-1005UBC), copied and adapted: sink drive per hardware/sch_contract.json and research/PINMAP.md, 2x 75R -> one 150R 0201, second column for LED1.\nCircuit: +3.3V -> LED -> 150R -> GPIO, the pin sinks (contract). Betaflight default polarity, low = on, no LEDx_INVERTED: LED0_PIN PA10 (GPIO10, green D5), LED1_PIN PA24 (GPIO24, blue D6).\nDatasheet check (XINGLIGHT XL-1005UGC / UBC, 0402): VF 2.7-3.3 / 2.6-3.4 V at 20 mA, IF max 20 mA, PD 70 mW, VR 5 V. At a few mA the InGaN VF is about 0.2-0.3 V lower (inferred), so with VOL <= 0.5 V at 4 mA drive (RP2350 DS) the LED current is about 0.5-5 mA, typ. 2-3 mA, hard ceiling (3.3 - 2.4) / 150R = 6 mA: LED, 0201 resistor (<= 5.4 mW of 50 mW) and GPIO (4 mA setting, 100 mA IOVSS sum) all inside their ratings; brightness at 1-3 mA is about 17-135 mcd green and 4-36 mcd blue (Iv scaled from 350-900 / 80-240 mcd at 20 mA), enough for an indicator. Reverse bias is 0 V when the pin drives high (IOVDD = +3.3V).\nReset state: RP2350 pads come up with the pull-down on (PDE = 1, 36-113 kOhm), so both LEDs may glow faintly (about 10-30 uA) until Betaflight drives the pins and in BOOTSEL mode. Accepted, cosmetic.\nPlacement (P5): bottom side, fc_core region (bom_plan); the R may sit at either end of the LED, slow signal (D33). Pins LED0/LED1 = root nets /LED0, /LED1 (RP2350A).\nP4 closed here: bom_plan R85/R86 'P4 checks brightness vs Vf' (above). P4-14 fields: RC0201FR-07150RL is a stocked Yageo RC_L part (Element14 4008725, RS 198-7568: 150R 1 % 50 mW 25 V); no LCSC number known, field left empty (contract open item A9-LCSC)."
 		(exclude_from_sim no)
 		(at 88.9 25.4 0)
@@
 			)
 		)
-		(property "Footprint" "lib:R_0201_0603Metric_W"
+		(property "Footprint" "lib:R_0201_0603Metric_L"
 			(at 66.04 60.96 0)
 			(hide yes)
@@
 			)
 		)
-		(property "Footprint" "lib:R_0201_0603Metric_W"
+		(property "Footprint" "lib:R_0201_0603Metric_L"
 			(at 45.72 60.96 0)
 			(hide yes)
@@
 	)
 	(symbol
-		(lib_id "power:+3V3")
+		(lib_id "power:+3.3V")
 		(at 45.72 40.64 0)
 		(unit 1)
@@
 		(in_pos_files no)
 		(dnp no)
-		(property "Reference" "#PWR236"
+		(property "Reference" "#PWR237"
 			(at 45.72 44.45 0)
 			(hide yes)
@@
 			)
 		)
-		(property "Value" "+3V3"
+		(property "Value" "+3.3V"
 			(at 45.72 37.084 0)
 			(show_name no)
@@
 			)
 		)
-		(property "Description" "Power symbol creates a global label with name \"+3V3\""
+		(property "Description" "Power symbol creates a global label with name \"+3.3V\""
 			(at 45.72 40.64 0)
 			(hide yes)
@@
 			(project "OpenAIO-Whoop"
 				(path "/2c3a7206-1e66-4d43-a02f-491225e20dd6/0a9dca22-7345-53f8-9367-07faa3e8899c"
-					(reference "#PWR236")
+					(reference "#PWR237")
 					(unit 1)
 				)
@@
 			)
 		)
-		(property "Footprint" "lib:LED_0402_1005Metric"
+		(property "Footprint" "lib:LED_0402_1005Metric_L"
 			(at 66.04 49.53 0)
 			(hide yes)
@@
 			)
 		)
-		(property "Footprint" "lib:LED_0402_1005Metric"
+		(property "Footprint" "lib:LED_0402_1005Metric_L"
 			(at 45.72 49.53 0)
 			(hide yes)
@@
 	)
 	(symbol
-		(lib_id "power:+3V3")
+		(lib_id "power:+3.3V")
 		(at 66.04 40.64 0)
 		(unit 1)
@@
 		(in_pos_files no)
 		(dnp no)
-		(property "Reference" "#PWR237"
+		(property "Reference" "#PWR238"
 			(at 66.04 44.45 0)
 			(hide yes)
@@
 			)
 		)
-		(property "Value" "+3V3"
+		(property "Value" "+3.3V"
 			(at 66.04 37.084 0)
 			(show_name no)
@@
 			)
 		)
-		(property "Description" "Power symbol creates a global label with name \"+3V3\""
+		(property "Description" "Power symbol creates a global label with name \"+3.3V\""
 			(at 66.04 40.64 0)
 			(hide yes)
@@
 			(project "OpenAIO-Whoop"
 				(path "/2c3a7206-1e66-4d43-a02f-491225e20dd6/0a9dca22-7345-53f8-9367-07faa3e8899c"
-					(reference "#PWR237")
+					(reference "#PWR238")
 					(unit 1)
 				)
