File: hardware/led.kicad_sch (KiCad schematic)
At the start: 4 parts

Commit message: Trim BOM to strictly needed parts, fill sourcing fields, fix library datasheets
Owner review 2026-10-11, schematic only (board not resynced).

Removed (17 parts): D1 TVS (clamps above every IC abs max), R2/R3/C5
INA186 input RC, U5 TPS22810 O4 switch with C16/C129/R9/R10/R87/D2
(VHD pad now on +5V_BST, as Matrix HD boards; HD_EN still holds the
analog VTX off via Q28, R11 kept), R67 selector (PA_VCC is +BATT),
TH1/R70 PA NTC and R84 (patched-ELRS only; GPIO37/GPIO4 no-connect),
C92 and C121 (beyond SX1281 / LP5912 datasheet decoupling).

Changed: D4 WS2812 VDD to +5V (3.5 V min); X3 TCXO pin 1 floating per
the YXC sheet; C122/C123/C134 4.7 uF 0402 -> 0201 GRM035R60J475ME15D.

Sourcing: LCSC numbers for 21 MPN lines (SKUBAAE010 has no listing);
every BOM part keeps MPN + Manufacturer for NextPCB.

Library: 16 unused lib symbols pruned; dead or HTML-only datasheet
links replaced with verified PDF URLs (RTC6705, SE5004L, FL2, X1,
EFM8BB51, BC857BM, FTC252012, HCS1206 shunt, Molex 53047).

Net-class patterns and contract entries for the removed nets dropped;
PINMAP ESP32 rows updated (GPIO36 is ADC1_CH0).

Validation: ERC 0 errors / 2 warnings (baseline); check_netlist 7 ok;
sch_integrate --check idempotent; check_conventions unchanged.

Co-Authored-By: Claude Opus 5.5 <noreply@anthropic.com>
Parts:
- R85, R86: LCSC (none) -> C295773
Changed lines of the file:
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@@
 			)
 		)
-		(property "LCSC" ""
+		(property "LCSC" "C295773"
 			(at 66.04 60.96 0)
 			(hide yes)
@@
 			)
 		)
-		(property "LCSC" ""
+		(property "LCSC" "C295773"
 			(at 45.72 60.96 0)
 			(hide yes)
@@
 		(in_pos_files no)
 		(dnp no)
-		(property "Reference" "#PWR236"
+		(property "Reference" "#PWR223"
 			(at 45.72 44.45 0)
 			(hide yes)
@@
 			(project "OpenAIO-Whoop"
 				(path "/2c3a7206-1e66-4d43-a02f-491225e20dd6/0a9dca22-7345-53f8-9367-07faa3e8899c"
-					(reference "#PWR236")
+					(reference "#PWR223")
 					(unit 1)
 				)
@@
 		(in_pos_files no)
 		(dnp no)
-		(property "Reference" "#PWR237"
+		(property "Reference" "#PWR224"
 			(at 66.04 44.45 0)
 			(hide yes)
@@
 			(project "OpenAIO-Whoop"
 				(path "/2c3a7206-1e66-4d43-a02f-491225e20dd6/0a9dca22-7345-53f8-9367-07faa3e8899c"
-					(reference "#PWR237")
+					(reference "#PWR224")
 					(unit 1)
 				)

Commit message: Footprint audit vs datasheets, 0201 lands to Murata minimum, schematic notes shortened
Footprints: 45 checked against their datasheets by group, no pin or
land errors. C/R/L_0201_..._L pad height 0.28 -> 0.30 (Murata GRM03
reflow table c >= 0.30); other lands already at least density per D109
and left unchanged. Land spec texts cleaned (sources, shared parts).

Schematic notes: 157 -> 152 items, 19.5k -> 9.7k characters, all
current (diode-OR, removed parts, RTC6705 filters, TX0/RX0).

check_footprint 107/107 lib specs PASS; ERC 0 errors / 2 warnings;
check_netlist 7 ok; sch_integrate --check clean. Board not synced.

Co-Authored-By: Claude Opus 5.5 <noreply@anthropic.com>
Other:
- note added: "STATUS LEDS"
- note removed: "status LEDs"
Changed lines of the file:
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@@
 		)
 	)
-	(text "status LEDs"
+	(text "STATUS LEDS"
 		(exclude_from_sim no)
 		(at 44.45 33.02 0)
@@
 		)
 	)
-	(text_box "Status LEDs from OpenFC-Lite-Mini: +3.3V -> LED -> 150R -> GPIO, the pin sinks (low = on, Betaflight default). LED0 = GPIO10 green D5, LED1 = GPIO24 blue D6.\nAbout 2-3 mA, ceiling 6 mA: LED, resistor and GPIO well inside ratings. The LEDs may glow faintly from the reset pull-downs until Betaflight drives the pins: cosmetic, accepted. Slow signal, R at either end (D33)."
+	(text_box "+3.3V -> LED -> 150R -> GPIO, the pin sinks (low = on). LED0 GPIO10 green, LED1 GPIO24 blue, about 2-3 mA.\nThe LEDs may glow faintly during reset: cosmetic."
 		(exclude_from_sim no)
 		(at 88.9 25.4 0)

Commit message: Every schematic symbol project-local (Device, power, Connector, Mechanical moved into lib)
tools/localise_symbols.py from OpenAIO. Netlist identical, ERC unchanged (0 errors, 24 warnings), every symbol, footprint and 3D model resolves inside the repo.

Co-Authored-By: Claude Opus 5.5 <noreply@anthropic.com>
Parts:
- D5, D6: symbol Device:LED -> lib:LED
- R85, R86: symbol Device:R -> lib:R
Changed lines of the file:
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@@
 	)
 	(symbol
-		(lib_id "Device:R")
+		(lib_id "lib:R")
 		(at 66.04 60.96 0)
 		(unit 1)
@@
 	)
 	(symbol
-		(lib_id "Device:R")
+		(lib_id "lib:R")
 		(at 45.72 60.96 0)
 		(unit 1)
@@
 	)
 	(symbol
-		(lib_id "power:+3.3V")
+		(lib_id "lib:+3.3V")
 		(at 45.72 40.64 0)
 		(unit 1)
@@
 	)
 	(symbol
-		(lib_id "Device:LED")
+		(lib_id "lib:LED")
 		(at 66.04 49.53 90)
 		(unit 1)
@@
 	)
 	(symbol
-		(lib_id "Device:LED")
+		(lib_id "lib:LED")
 		(at 45.72 49.53 90)
 		(unit 1)
@@
 	)
 	(symbol
-		(lib_id "power:+3.3V")
+		(lib_id "lib:+3.3V")
 		(at 66.04 40.64 0)
 		(unit 1)
