File: hardware/rp2350a.kicad_sch (KiCad schematic)
At the start: 0 parts

Commit message: wip: schematic sheets in progress
Co-Authored-By: Claude Opus 5.5 <noreply@anthropic.com>
Claude-Session: https://claude.ai/code/session_01RFaS5jnC9tnPam9GBgmGnG
Parts:
- added C42, C43: 15pF, lib:C_0201_0603Metric_W, symbol Device:C
- added C44, C45, C46, C47, C48, C49, C50, C51, C52, C54, C59, C60: 100nF, lib:C_0201_0603Metric_W, symbol Device:C
- added C56, C57, C58: 4.7uF, lib:C_0402_1005Metric_W, symbol Device:C
- added L2: 3.3uH, lib:IND-SMD_L2.0-W1.6_AOTA-B201610S3R3-101-T_Dense, symbol OpenDrone:AOTA-B201610S3R3-101-T
- added Q26: AP1606, lib:DFN-3L_L1.0-W0.6-P0.65-BR_W, symbol OpenDrone:AP1606
- added R40, R44, R47: 1k, lib:R_0201_0603Metric_W, symbol Device:R
- added R41, R42, R43: 27R, lib:R_0201_0603Metric_W, symbol Device:R
- added R45, R46: 10k, lib:R_0201_0603Metric_W, symbol Device:R
- added R48: 100k, lib:R_0201_0603Metric_W, symbol Device:R
- added TP12: CLK, lib:TestPoint_Via_D0.35mm_Drill0.2mm, symbol Connector:TestPoint
- added TP13: DIO, lib:TestPoint_Via_D0.35mm_Drill0.2mm, symbol Connector:TestPoint
- added TP9: FCB, lib:TestPoint_Via_D0.35mm_Drill0.2mm, symbol Connector:TestPoint
- added U10: RP2354A, lib:QFN-60_L7.0-W7.0-P0.40-TL-EP3.4_Dense, symbol OpenDrone:RP2354A
- added X1: 12MHz 10pF, lib:CRYSTAL-SMD_4P-L2.5-W2.0-BL-A_Dense, symbol Device:Crystal_GND24
Connections:
- new net: L2.2, U10.48 (VREG_LX)
- new net +1V1: C50.1, C51.1, C52.1, C56.1, L2.1, U10.23 (DVDD), U10.39 (DVDD), U10.50 (VREG_FB), U10.6 (DVDD)
- new net +3V3: C44.1, C45.1, C46.1, C47.1, C48.1, C49.1, C54.1, C58.1, R41.1, U10.1 (IOVDD), U10.11 (IOVDD), U10.20 (IOVDD), U10.26 (RUN), U10.30 (IOVDD), U10.38 (IOVDD), U10.44 (ADC_AVDD), U10.45 (IOVDD), U10.49 (VREG_VIN), U10.53 (USB_OTP_VDD), U10.54 (QSPI_IOVDD)
- new net +BATT: R45.2
- new net ADC_CURR: C60.1, R47.2, U10.42 (GPIO28_ADC2)
- new net ADC_VBAT: C59.2, R45.1, R46.2, U10.43 (GPIO29_ADC3)
- new net BEEPER: Q26.1 (G), R48.2, U10.28 (GPIO17)
- new net BUZZER-: Q26.3 (D)
- new net CURR_SENSE: R47.1
- new net FC_BOOT: R44.2, TP9.1
- new net FLASH_CS: U10.33 (GPIO21)
- new net GND: C42.2, C43.2, C44.2, C45.2, C46.2, C47.2, C48.2, C49.2, C50.2, C51.2, C52.2, C54.2, C56.2, C57.2, C58.2, C59.1, C60.2, Q26.2 (S), R46.1, R48.1, U10.47 (VREG_PGND), U10.61 (EP), X1.2 (G), X1.4 (G)
- new net GYRO_CLKIN: U10.9 (GPIO6)
- new net GYRO_CS: U10.17 (GPIO13)
- new net GYRO_INT: U10.13 (GPIO9)
- new net HD_EN: U10.41 (GPIO27_ADC1)
- new net LED0: U10.10 (GPIO7)
- new net LED1: U10.40 (GPIO26_ADC0)
- new net LED_STRIP: U10.12 (GPIO8)
- new net MOTOR1: U10.37 (GPIO25)
- new net MOTOR2: U10.36 (GPIO24)
- new net MOTOR3: U10.35 (GPIO23)
- new net MOTOR4: U10.34 (GPIO22)
- new net OSD_EN: U10.19 (GPIO15)
- new net OSD_SYNC: U10.27 (GPIO16)
- new net OSD_W: U10.18 (GPIO14)
- new net PIOUART0_RX: U10.5 (GPIO3)
- new net PIOUART0_TX: U10.4 (GPIO2)
- new net QSPI_SS: R44.1, U10.60 (QSPI_SS)
- new net SPI0_MISO: U10.32 (GPIO20)
- new net SPI0_MOSI: U10.31 (GPIO19)
- new net SPI0_SCK: U10.29 (GPIO18)
- new net SPI1_MISO: U10.16 (GPIO12)
- new net SPI1_MOSI: U10.15 (GPIO11)
- new net SPI1_SCK: U10.14 (GPIO10)
- new net SWCLK: TP12.1, U10.24 (SWCLK)
- new net SWDIO: TP13.1, U10.25 (SWDIO)
- new net U10_USB_DM: R43.2, U10.51 (USB_DM)
- new net U10_USB_DP: R42.1, U10.52 (USB_DP)
- new net UART0_RX: U10.3 (GPIO1)
- new net UART0_TX: U10.2 (GPIO0)
- new net UART1_RX: U10.8 (GPIO5)
- new net UART1_TX: U10.7 (GPIO4)
- new net USB_D_N: R43.1
- new net USB_D_P: R42.2
- new net VREG_AVDD: C57.1, R41.2, U10.46 (VREG_AVDD)
- new net XIN: C42.1, U10.21 (XIN), X1.1
- new net XOUT: R40.2, U10.22 (XOUT)
- new net XOUT_X: C43.1, R40.1, X1.3
- no-connect marks 0 -> 5
Other:
- note added: "Boot strap + SWD test vias"
- note added: "Crystal per datasheet. 10pF loading = 2x 15pF in series + ~2.5pF stray"
- note added: "HD line PINIO1: high = O4 on, analog VTX off"
- note added: "PIO0 bidir. DShot to the EFM8s (2.4k at the EFM8)"
- note added: "PIO2 framebuffer OSD: W, EN, SYNC consecutive"
- note added: "RP2354A: Smaller variant with integrated flash (2MB)"
- note added: "WS2812 pad LED, driven direct (F1, BR-04)"
- note added: "blackbox SPI0 (FLASH_CS pull-up R50 there)"
- note added: "buzzer with N-MOS low side switch"
- note added: "current sense RC, 1.6 kHz"
- note added: "decoupling caps, place close to IC, one is enough when 2 pins are next to each other"
- note added: "for CRSF receiver (ESP32 ELRS, UART0)"
- note added: "for MSP DisplayPort: DJI O4 Lite TX1/RX1"
- note added: "for external: user pads TP0/RP0 (PIO1, 8N1)"
- note added: "gyro CLKIN (ICM-42688-P only)"
- note added: "gyro SPI1 (IMU; GYRO_CS pull-up R49 there)"
- note added: "in-package flash on QSPI: SD0-SD3, SCLK no-connect"
- note added: "status LEDs (LED sheet, sinking)"
- note added: "vbat sense, 1/2 scale"

Commit message: wip: schematic integration in progress (saved after container restart)
Co-Authored-By: Claude Opus 5.5 <noreply@anthropic.com>
Claude-Session: https://claude.ai/code/session_01RFaS5jnC9tnPam9GBgmGnG
Parts:
- added C134: 4.7uF, lib:C_0402_1005Metric_W, symbol Device:C
- L2: symbol OpenDrone:AOTA-B201610S3R3-101-T -> lib:AOTA-B201610S3R3-101-T
- Q26: symbol OpenDrone:AP1606 -> lib:AP1606
- U10: symbol OpenDrone:RP2354A -> lib:RP2354A
Connections:
- net +1V1: now also C134.1
- net GND: now also C134.2
- net VREG_LX: now reaches L2.2, U10.48 (VREG_LX)

Commit message: schematic: integrated (ERC 0 errors / 2 justified warnings; check_netlist 7/7; conventions 0 FAIL; visual 0 hits; 268/268 refs match bom_plan; FC+RX pin maps match PINMAP)
Co-Authored-By: Claude Opus 5.5 <noreply@anthropic.com>
Claude-Session: https://claude.ai/code/session_01RFaS5jnC9tnPam9GBgmGnG
Parts:
- X1: value 12MHz 10pF -> 12MHz; footprint lib:CRYSTAL-SMD_4P-L2.5-W2.0-BL-A_Dense -> lib:CRYSTAL-SMD_4P-L3.2-W2.5-BL_Dense; LCSC C2896601 -> C20625731; MPN X252012MMB4SI-24 -> ABM8-272-T3; Manufacturer YXC -> Abracon

Commit message: hardware: floorplan v3 review pass (RX RF corner blocker fixed; majors listed in FLOORPLAN.md Open)
Co-Authored-By: Claude Opus 5.5 <noreply@anthropic.com>
Claude-Session: https://claude.ai/code/session_01RFaS5jnC9tnPam9GBgmGnG
Changed lines of the file:
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@@
 		)
 	)
-	(text_box "P4-11 power-up and 5 V-tolerant pads (PINMAP 4.5, F16; RP2350 DS Table 1433): an FT pad takes <= 3.63 V while IOVDD is 0-1.8 V (4.2 V at 2.5 V, 5.5 V at 3.3 V); the ADC pads GPIO26-29 take <= IOVDD + 0.5 V.\n- MOTOR1-4 (GPIO25-22, FT), battery first: each EFM8 weak pull-up (70-220 kOhm to VDD = cell) reaches the pad through its 2.4k before +3V3 is up (boost soft start + LP5912 ramp, about 1-2 ms). Worst case 4.35 V open circuit = 0.72 V over 3.63 V, from >= 72 kOhm (<= 60 uA). Matrix parity (G473 FT pins ~4 V at VDD 0). V9 scopes it; fallback (F16): 3.3 V-domain clamp or DShot-path enable.\n- ADC_VBAT (GPIO29): R45/R46 put up to 2.18 V on the pad from 5 kOhm while IOVDD < 1.7 V, so the pad clamp to IOVDD conducts <= 0.3 mA during the ramp. House + Matrix parity; V9 scope.\n- HD_EN (GPIO27): R11 2.4k + the BAS16LD from O4_EN (<= 90 uA) hold it at <= 0.22 V before and during reset: inside IOVDD + 0.5 V and below the AP1606 HD-gate Vgs(th) min 0.4 V (P4-4); driven high it is >= 2.62 V (VOH, 1.4 mA into R11) over Vgs(th) max 1.2 V.\n- UART0, SPI0/1, gyro, OSD, CURR_SENSE: every driver is on +3V3 = IOVDD, no excursion. UART1 TX1/RX1: the O4 is fed only through U5 (needs HD_EN high), none. USB D+/D-: the host drives only after the device pull-up.\n- PIOUART0 pads TP0/RP0: a peripheral on the 5V pads is up before IOVDD: 3.3 V logic only (README); a 5 V TX would exceed 3.63 V at power-up."
+	(text_box "P4-11 power-up and 5 V-tolerant pads (PINMAP 4.5, F16; RP2350 DS Table 1433): an FT pad takes <= 3.63 V while IOVDD is 0-1.8 V (4.2 V at 2.5 V, 5.5 V at 3.3 V); the ADC pads GPIO26-29 take <= IOVDD + 0.5 V.\n- MOTOR1-4 (GPIO25-22, FT), battery first: each EFM8 weak pull-up (70-220 kOhm to VDD = cell) reaches the pad through its 2.4k before +3V3 is up (boost soft start + LP5912 ramp, about 1-2 ms). Worst case 4.35 V open circuit = 0.72 V over 3.63 V, from >= 72 kOhm (<= 60 uA). Matrix parity (G473 FT pins ~4 V at VDD 0). V9 scopes it; fallback (F16): 3.3 V-domain clamp or DShot-path enable.\n- ADC_VBAT (GPIO29): R45/R46 put up to 2.18 V on the pad from 5 kOhm while IOVDD < 1.7 V, so the pad clamp to IOVDD conducts <= 0.3 mA during the ramp. House + Matrix parity; V9 scope.\n- HD_EN (GPIO27): R11 2.4k + the BAS16LD from O4_EN (<= 90 uA) hold it at <= 0.22 V before and during reset: inside IOVDD + 0.5 V and below the AP1606 HD-gate Vgs(th) min 0.4 V (P4-4); driven high it is >= 2.62 V (VOH, 1.4 mA into R11) over Vgs(th) max 1.2 V.\n- UART0, SPI0/1, gyro, OSD, CURR_SENSE: every driver is on +3V3 = IOVDD, no excursion. UART1 TX1/RX1: the O4 is fed only through U5 (needs HD_EN high), none. USB D+/D-: the host drives only after the device pull-up.\n- PIOUART0 pads TP0/RP0, and TX1/RX1 used as the second hardware UART in analog builds (IO-SET row 8): a peripheral on the 5V pads is up before IOVDD: 3.3 V logic only (README); a 5 V TX on RP0 or RX1 (GPIO5) would exceed 3.63 V at power-up."
 		(exclude_from_sim no)
 		(at 424.18 208.28 0)

Commit message: wip: routing prep (zones and via fields) and schematic review round 4
Co-Authored-By: Claude Opus 5.5 <noreply@anthropic.com>
Claude-Session: https://claude.ai/code/session_01RFaS5jnC9tnPam9GBgmGnG
Changed lines of the file:
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@@
 		)
 	)
-	(text_box "RP2350 1.1V DC-DC SMPS: follow the datasheet placement. RP2350 DS 6.3.8 (binding): C58 = CIN at VREG_VIN, C56 = COUT on +1V1 with VREG_FB taken from the C56 pad (not under L2); C58, L2 and C56 on the U10 side, smallest hot loops; CIN/COUT GND to VREG_PGND at one point with 2 vias; no copper under L2 / VREG_LX on the next layer. L2 AOTA-B201610S3R3 is polarity-marked: orientation as DS Fig. 23/25 (pin 2 = VREG_LX as on the flown house board). R41 27R + C57 4.7 uF filter VREG_AVDD (1.25 kHz, BR-21; 3.135-3.63 V); C57 gets its own GND via to the EP. DS: CIN >= 4.7 uF, COUT 4.7 uF +/-20 %; C134 = the 2nd 4.7 uF on +1V1 that DS 6.3.8 recommends at DVDD pin 23 (fitted per the 2026-10-09 ruling, house board fits two): place it at pin 23."
+	(text_box "RP2350 1.1V DC-DC SMPS: follow the datasheet placement. RP2350 DS 6.3.8 (binding): C58 = CIN at VREG_VIN, C56 = COUT on +1V1 with VREG_FB taken from the C56 pad (not under L2); C58, L2 and C56 on the U10 side, smallest hot loops; CIN/COUT GND to VREG_PGND at one point with 2 vias; no copper under L2 / VREG_LX on the next layer. L2 AOTA-B201610S3R3 is polarity-marked: orientation as DS Fig. 26 / 28 (pin 2 = VREG_LX as on the flown house board). P5 condition (tools/check_p5_conditions.py SMPS): C58, L2, C56 and C57 on U10's side within 3 mm of pins 49 / 48 / 50 / 46. R41 27R + C57 4.7 uF filter VREG_AVDD (1.25 kHz, BR-21; 3.135-3.63 V); C57 gets its own GND via to the EP. DS: CIN >= 4.7 uF, COUT 4.7 uF +/-20 %; C134 = the 2nd 4.7 uF on +1V1 that DS 6.3.8 recommends at DVDD pin 23 (fitted per the 2026-10-09 ruling, house board fits two): place it at pin 23."
 		(exclude_from_sim no)
 		(at 223.52 292.1 0)

Commit message: schematic: review complete (4 rounds; U20 pin 1 to GND, footprint filters fixed, TPS22810DRVR, R54 270R); ERC 0 errors, check_netlist 7/7; D85-D87
Co-Authored-By: Claude Opus 5.5 <noreply@anthropic.com>
Claude-Session: https://claude.ai/code/session_01RFaS5jnC9tnPam9GBgmGnG
Changed lines of the file:
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@@
 		)
 	)
-	(text_box "P4-11 power-up and 5 V-tolerant pads (PINMAP 4.5, F16; RP2350 DS Table 1433): an FT pad takes <= 3.63 V while IOVDD is 0-1.8 V (4.2 V at 2.5 V, 5.5 V at 3.3 V); the ADC pads GPIO26-29 take <= IOVDD + 0.5 V.\n- MOTOR1-4 (GPIO25-22, FT), battery first: each EFM8 weak pull-up (70-220 kOhm to VDD = cell) reaches the pad through its 2.4k before +3V3 is up (boost soft start + LP5912 ramp, about 1-2 ms). Worst case 4.35 V open circuit = 0.72 V over 3.63 V, from >= 72 kOhm (<= 60 uA). Matrix parity (G473 FT pins ~4 V at VDD 0). V9 scopes it; fallback (F16): 3.3 V-domain clamp or DShot-path enable.\n- ADC_VBAT (GPIO29): R45/R46 put up to 2.18 V on the pad from 5 kOhm while IOVDD < 1.7 V, so the pad clamp to IOVDD conducts <= 0.3 mA during the ramp. House + Matrix parity; V9 scope.\n- HD_EN (GPIO27): R11 2.4k + the BAS16LD from O4_EN (<= 90 uA) hold it at <= 0.22 V before and during reset: inside IOVDD + 0.5 V and below the AP1606 HD-gate Vgs(th) min 0.4 V (P4-4); driven high it is >= 2.62 V (VOH, 1.4 mA into R11) over Vgs(th) max 1.2 V.\n- UART0, SPI0/1, gyro, OSD, CURR_SENSE: every driver is on +3V3 = IOVDD, no excursion. UART1 TX1/RX1: the O4 is fed only through U5 (needs HD_EN high), none. USB D+/D-: the host drives only after the device pull-up.\n- PIOUART0 pads TP0/RP0, and TX1/RX1 used as the second hardware UART in analog builds (IO-SET row 8): a peripheral on the 5V pads is up before IOVDD: 3.3 V logic only (README); a 5 V TX on RP0 or RX1 (GPIO5) would exceed 3.63 V at power-up."
+	(text_box "P4-11 power-up and 5 V-tolerant pads (PINMAP 4.5, F16; RP2350 DS Table 1433): an FT pad takes <= 3.63 V while IOVDD is 0-1.8 V (4.2 V at 2.5 V, 5.5 V at 3.3 V); the ADC pads GPIO26-29 take <= IOVDD + 0.5 V.\n- MOTOR1-4 (GPIO25-22, FT), battery first: each EFM8 weak pull-up (70-220 kOhm to VDD = cell) reaches the pad through its 2.4k before +3V3 is up (boost soft start + LP5912 ramp, about 1-2 ms). Worst case 4.35 V open circuit = 0.72 V over 3.63 V, from >= 72 kOhm (<= 60 uA). Matrix parity (G473 FT pins ~4 V at VDD 0). V9 scopes it; fallback (F16): 3.3 V-domain clamp or DShot-path enable.\n- ADC_VBAT (GPIO29): R45/R46 put up to 2.18 V on the pad from 5 kOhm while IOVDD < 1.7 V, so the pad clamp to IOVDD conducts <= 0.3 mA during the ramp. House + Matrix parity; V9 scope.\n- HD_EN (GPIO27): R11 2.4k + the BAS16LD from O4_EN (<= 90 uA) hold it at <= 0.22 V before and during reset: inside IOVDD + 0.5 V and below the AP1606 HD-gate Vgs(th) min 0.4 V at 25 C (P4-4; about 0.25 V at 85 C, -2.5 mV/K: a hot low-Vth part may hold the analog VTX off until PINIO1 is driven low, R68 47k, V9 hot-soak boot check); driven high it is >= 2.62 V (VOH, 1.4 mA into R11) over Vgs(th) max 1.2 V.\n- UART0, SPI0/1, gyro, OSD, CURR_SENSE: every driver is on +3V3 = IOVDD, no excursion. UART1 TX1/RX1: the O4 is fed only through U5 (needs HD_EN high), none. USB D+/D-: the host drives only after the device pull-up.\n- PIOUART0 pads TP0/RP0, and TX1/RX1 used as the second hardware UART in analog builds (IO-SET row 8): a peripheral on the 5V pads is up before IOVDD: 3.3 V logic only (README); a 5 V TX on RP0 or RX1 (GPIO5) would exceed 3.63 V at power-up."
 		(exclude_from_sim no)
 		(at 424.18 208.28 0)

Commit message: wip: v4 prep in progress (D89 UART pad removal, D93 3D model fixes, Wi-Fi antenna research)
Snapshot of running workflows; final numbers follow when each verifies.

Co-Authored-By: Claude Opus 5.5 <noreply@anthropic.com>
Claude-Session: https://claude.ai/code/session_01RFaS5jnC9tnPam9GBgmGnG
Connections:
- net PIOUART0_RX: no longer names the net of U10.5 (GPIO3)
- net PIOUART0_TX: no longer names the net of U10.4 (GPIO2)
- no-connect marks 5 -> 7
Other:
- note added: "GPIO2/3 spare, no-connect (D89)"
- note removed: "for external: user pads TP0/RP0 (PIO1, 8N1)"
