File: hardware/rp2350a.kicad_sch (KiCad schematic)
At the start: 32 parts, among them Q26 AP1606, U10 RP2354A, X1 12MHz

Commit message: Trim BOM to strictly needed parts, fill sourcing fields, fix library datasheets
Owner review 2026-10-11, schematic only (board not resynced).

Removed (17 parts): D1 TVS (clamps above every IC abs max), R2/R3/C5
INA186 input RC, U5 TPS22810 O4 switch with C16/C129/R9/R10/R87/D2
(VHD pad now on +5V_BST, as Matrix HD boards; HD_EN still holds the
analog VTX off via Q28, R11 kept), R67 selector (PA_VCC is +BATT),
TH1/R70 PA NTC and R84 (patched-ELRS only; GPIO37/GPIO4 no-connect),
C92 and C121 (beyond SX1281 / LP5912 datasheet decoupling).

Changed: D4 WS2812 VDD to +5V (3.5 V min); X3 TCXO pin 1 floating per
the YXC sheet; C122/C123/C134 4.7 uF 0402 -> 0201 GRM035R60J475ME15D.

Sourcing: LCSC numbers for 21 MPN lines (SKUBAAE010 has no listing);
every BOM part keeps MPN + Manufacturer for NextPCB.

Library: 16 unused lib symbols pruned; dead or HTML-only datasheet
links replaced with verified PDF URLs (RTC6705, SE5004L, FL2, X1,
EFM8BB51, BC857BM, FTC252012, HCS1206 shunt, Molex 53047).

Net-class patterns and contract entries for the removed nets dropped;
PINMAP ESP32 rows updated (GPIO36 is ADC1_CH0).

Validation: ERC 0 errors / 2 warnings (baseline); check_netlist 7 ok;
sch_integrate --check idempotent; check_conventions unchanged.

Co-Authored-By: Claude Opus 5.5 <noreply@anthropic.com>
Parts:
- C134: footprint lib:C_0402_1005Metric_L -> lib:C_0201_0603Metric_L; LCSC C23733 -> C335103; MPN CL05A475MP5NRNC -> GRM035R60J475ME15D; Manufacturer Samsung Electro-Mechanics -> Murata
- R41, R42, R43: LCSC (none) -> C273268
- R44, R47: LCSC (none) -> C138165

Commit message: Library: X1 land from the YSO110TR sheet, symbol default footprints, orphan specs, LIBRARY.md counts
New lib:OSC-SMD_4P-L2.0-W1.6-BL_YXC_YSO110TR_Dense for X1 (check_footprint
PASS); 26 lib symbols now default to the footprint the schematic places;
9 orphan land specs and an unused 3D file removed; LIBRARY.md summary
regenerated with the _L/_Dense/_W variant table.

check_footprint 106/106 PASS; ERC 0 errors; check_netlist 7 ok.

Co-Authored-By: Claude Opus 5.5 <noreply@anthropic.com>
Parts:
- X1: footprint lib:OSC-SMD_4P-L2.0-W1.6-BL_TXC_7Z_Dense -> lib:OSC-SMD_4P-L2.0-W1.6-BL_YXC_YSO110TR_Dense
Changed lines of the file:
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@@
 			)
 		)
-		(property "Footprint" "lib:OSC-SMD_4P-L2.0-W1.6-BL_TXC_7Z_Dense"
+		(property "Footprint" "lib:OSC-SMD_4P-L2.0-W1.6-BL_YXC_YSO110TR_Dense"
 			(at 143.51 172.72 0)
 			(hide yes)

Commit message: Footprint audit vs datasheets, 0201 lands to Murata minimum, schematic notes shortened
Footprints: 45 checked against their datasheets by group, no pin or
land errors. C/R/L_0201_..._L pad height 0.28 -> 0.30 (Murata GRM03
reflow table c >= 0.30); other lands already at least density per D109
and left unchanged. Land spec texts cleaned (sources, shared parts).

Schematic notes: 157 -> 152 items, 19.5k -> 9.7k characters, all
current (diode-OR, removed parts, RTC6705 filters, TX0/RX0).

check_footprint 107/107 lib specs PASS; ERC 0 errors / 2 warnings;
check_netlist 7 ok; sch_integrate --check clean. Board not synced.

Co-Authored-By: Claude Opus 5.5 <noreply@anthropic.com>
Other:
- note added: "12 MHz CMOS oscillator on XIN, XOUT open"
- note added: "RP2354A: in-package flash"
- note added: "decoupling caps close to the IC"
- note removed: "12 MHz CMOS oscillator on XIN, XOUT open (D100)"
- note removed: "RP2354A: Smaller variant with integrated flash (2MB)"
- note removed: "decoupling caps, place close to IC, one is enough when 2 pins are next to each other"
Changed lines of the file:
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@@
 		)
 	)
-	(text "decoupling caps, place close to IC, one is enough when 2 pins are next to each other"
+	(text "decoupling caps close to the IC"
 		(exclude_from_sim no)
 		(at 177.8 71.12 0)
@@
 		)
 	)
-	(text "RP2354A: Smaller variant with integrated flash (2MB)"
+	(text "RP2354A: in-package flash"
 		(exclude_from_sim no)
 		(at 199.644 27.686 0)
@@
 		)
 	)
-	(text "12 MHz CMOS oscillator on XIN, XOUT open (D100)"
+	(text "12 MHz CMOS oscillator on XIN, XOUT open"
 		(exclude_from_sim no)
 		(at 145.415 148.59 0)
@@
 		)
 	)
-	(text_box "GPIO map (D111, placement V4_B4; research/PINMAP.md):\nSPI0 blackbox GPIO0 MISO / 2 SCK / 3 MOSI, FLASH_CS GPIO1. SPI1 gyro GPIO11 MOSI / 12 MISO / 14 SCK, GYRO_CS 15, GYRO_INT 7, GYRO_CLKIN 13.\nUART1 GPIO8/9 = CRSF to the ESP32; UART0 GPIO16/17 = TX1/RX1 pads (O4 MSP, D89).\nDShot MOTOR1-4 GPIO4/6/18/20 (PIO0). LED_STRIP 5, LED0 10, LED1 24, BEEPER 25. HD_EN 19 (PINIO1, high = O4 on). OSD W/EN/SYNC 21/22/23 (PIO2). ADC_CURR 26, ADC_VBAT 27. GPIO28/29 no-connect."
+	(text_box "SPI0 blackbox GPIO0-3. SPI1 gyro 11/12/14, CS 15, INT 7, CLKIN 13. UART1 8/9 CRSF, UART0 16/17 TX0/RX0 pads.\nDShot 4/6/18/20. LED 5/10/24, BEEPER 25, HD_EN 19, OSD 21-23, ADC 26/27, GPIO28/29 NC."
 		(exclude_from_sim no)
 		(at 353.06 129.54 0)
@@
 		)
 	)
-	(text_box "R44 1k QSPI_SS -> FC_BOOT: the shared button SW1 (RX sheet, D65) pulls it low through D8, low at reset = BOOTSEL. Keep the QSPI_SS-to-R44 stub <= 1 mm.\nTP9 FCB, TP12 SWCLK, TP13 SWDIO: filled test vias (D67), out of the BOM."
+	(text_box "R44 1k QSPI_SS -> FC_BOOT: SW1 (RX sheet) pulls it low through D8 = BOOTSEL. Keep the QSPI_SS-to-R44 stub <= 1 mm.\nTP9, TP12, TP13: filled test vias."
 		(exclude_from_sim no)
 		(at 144.78 192.405 0)
@@
 		)
 	)
-	(text_box "100 nF X6S 0201 per supply pin: DVDD C50-C52, IOVDD C44-C48; C49 at ADC_AVDD 44 (also IOVDD 45), C54 <= 1 mm from QSPI_IOVDD 54 (also USB_OTP_VDD 53)."
+	(text_box "100 nF 0201 per supply pin; C49 at ADC_AVDD 44, C54 <= 1 mm from QSPI_IOVDD 54."
 		(exclude_from_sim no)
 		(at 91.44 73.66 0)
@@
 		)
 	)
-	(text_box "RP2350A sheet, copied block by block from OpenFC-Lite-Mini rp2350a (flown Rev2). Changes: USB on J31 (PADS) with 27R R42/R43 here (D52); no I2C pull-ups, no WS2812 inverter; LEDs on the LED sheet; boot via R44 + FC_BOOT; SWD on test vias (D67); 12 MHz CMOS oscillator (D100); GPIO map D111. Betaflight config: PINMAP 5."
-		(exclude_from_sim no)
-		(at 424.18 99.06 0)
-		(size 81.28 15.24)
-		(margins 0.9525 0.9525 0.9525 0.9525)
-		(stroke
-			(width -0.0001)
-			(type solid)
-		)
-		(fill
-			(type none)
-		)
-		(effects
-			(font
-				(size 1.27 1.27)
-			)
-			(justify left top)
-		)
-	)
-	(text_box "X1 12 MHz CMOS oscillator drives XIN (pin 21); XOUT stays open, no trace (D99, D100 replace the D78 crystal). C42 at X1 VDD; X1 within 3 mm of pin 21."
+	(text_box "X1 12 MHz CMOS oscillator on XIN (pin 21), XOUT open. C42 at X1 VDD; X1 within 3 mm of pin 21."
 		(exclude_from_sim no)
 		(at 93.98 150.495 0)
@@
 		)
 	)
-	(text_box "R42/R43 27R within 1-2 mm of pins 52/51. USB_D_P/N: 90 Ohm pair over solid GND, length-matched (D33)."
+	(text_box "R42/R43 27R within 1-2 mm of pins 52/51. USB_D_P/N: 90 Ohm pair over solid GND, length-matched."
 		(exclude_from_sim no)
 		(at 198.12 104.14 0)
@@
 		)
 	)
-	(text_box "Q26 AP1606 low-side buzzer switch (from OpenFC-Lite-Mini): GPIO25 high = on (BEEPER_INVERTED, active buzzer); R48 100k holds it off through reset. BZ- pad on PADS."
+	(text_box "Q26 AP1606 buzzer low-side switch: GPIO25 high = on. R48 100k holds it off through reset."
 		(exclude_from_sim no)
 		(at 387.35 78.74 0)
@@
 		)
 	)
-	(text_box "1.1 V SMPS: follow RP2350 DS 6.3.8 placement. C58 CIN, L2, C56 COUT on U10's side within 3 mm of pins 49/48/50/46, VREG_FB from the C56 pad, one-point GND to VREG_PGND, no copper under L2 on the next layer. L2 is polarity-marked (pin 2 = VREG_LX). C134 = 2nd 4.7 uF at DVDD pin 23. R41 + C57 filter VREG_AVDD."
+	(text_box "1.1 V SMPS per RP2350 DS 6.3.8: C58, L2, C56 within 3 mm of pins 49/48/50/46; VREG_FB from the C56 pad, one-point GND to VREG_PGND, no copper under L2 on the next layer.\nL2 pin 2 = VREG_LX; C134 4.7 uF at DVDD pin 23."
 		(exclude_from_sim no)
 		(at 223.52 215.9 0)
@@
 		)
 	)
-	(text_box "Power-up and 5 V-tolerant pads (PINMAP 4.5, F16): an FT pad takes <= 3.63 V while IOVDD is off.\n- MOTOR1-4: the EFM8 pull-ups reach the pads through 2.4k before +3.3V (<= 60 uA, current-limited); Matrix parity, V9 scope.\n- HD_EN (GPIO19): R11 2.4k holds it low through reset, so the O4 stays off and the analog VTX on (V9 hot-soak boot check).\n- TX1/RX1 as the free UART (D89): 3.3 V peripherals only; a 5 V TX would exceed 3.63 V at power-up.\n- GPIO28/29 spare, no-connect (D111 map)."
+	(text_box "Power-up: FT pads take <= 3.63 V while IOVDD is off. MOTOR1-4 pull-ups reach the pads through 2.4k (<= 60 uA); R11 holds HD_EN low.\nTX0/RX0: 3.3 V peripherals only."
 		(exclude_from_sim no)
 		(at 424.18 132.08 0)
@@
 		)
 	)
-	(text_box "VBAT: R45/R46 10k/10k, 4.35 V -> 2.18 V on GPIO27 (ADC1), vbat_scale 200/100. CURR: R47 1k + C60 100 nF on GPIO26 (ADC0), ibata_scale 500."
+	(text_box "VBAT: R45/R46 10k/10k, 4.35 V -> 2.18 V on GPIO27. CURR: R47 1k + C60 100 nF on GPIO26."
 		(exclude_from_sim no)
 		(at 91.44 135.255 0)
