File: hardware/pads.kicad_sch (KiCad schematic)
At the start: 21 parts, among them J10 M3, J13 M4, J20 LED, J21 5V, J22 BZ-, J23 CAM, J24 5V, J25 GND, J26 VHD, J27 GND, J28 TX1, J29 RX1, J31 USB, J32 CAM, J33 GND, J4 M1, J7 M2

Commit message: Trim BOM to strictly needed parts, fill sourcing fields, fix library datasheets
Owner review 2026-10-11, schematic only (board not resynced).

Removed (17 parts): D1 TVS (clamps above every IC abs max), R2/R3/C5
INA186 input RC, U5 TPS22810 O4 switch with C16/C129/R9/R10/R87/D2
(VHD pad now on +5V_BST, as Matrix HD boards; HD_EN still holds the
analog VTX off via Q28, R11 kept), R67 selector (PA_VCC is +BATT),
TH1/R70 PA NTC and R84 (patched-ELRS only; GPIO37/GPIO4 no-connect),
C92 and C121 (beyond SX1281 / LP5912 datasheet decoupling).

Changed: D4 WS2812 VDD to +5V (3.5 V min); X3 TCXO pin 1 floating per
the YXC sheet; C122/C123/C134 4.7 uF 0402 -> 0201 GRM035R60J475ME15D.

Sourcing: LCSC numbers for 21 MPN lines (SKUBAAE010 has no listing);
every BOM part keeps MPN + Manufacturer for NextPCB.

Library: 16 unused lib symbols pruned; dead or HTML-only datasheet
links replaced with verified PDF URLs (RTC6705, SE5004L, FL2, X1,
EFM8BB51, BC857BM, FTC252012, HCS1206 shunt, Molex 53047).

Net-class patterns and contract entries for the removed nets dropped;
PINMAP ESP32 rows updated (GPIO36 is ADC1_CH0).

Validation: ERC 0 errors / 2 warnings (baseline); check_netlist 7 ok;
sch_integrate --check idempotent; check_conventions unchanged.

Co-Authored-By: Claude Opus 5.5 <noreply@anthropic.com>
Connections:
- net +5V_HD renamed +5V_BST
Changed lines of the file:
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@@
 		(in_pos_files no)
 		(dnp no)
-		(property "Reference" "#PWR241"
+		(property "Reference" "#PWR228"
 			(at 30.48 133.35 0)
 			(hide yes)
@@
 			(project "OpenAIO-Whoop"
 				(path "/2c3a7206-1e66-4d43-a02f-491225e20dd6/8d214749-72cf-5803-99b7-260f0c3f1838"
-					(reference "#PWR241")
+					(reference "#PWR228")
 					(unit 1)
 				)
@@
 		(in_pos_files no)
 		(dnp no)
-		(property "Reference" "#PWR239"
+		(property "Reference" "#PWR226"
 			(at 367.03 49.53 0)
 			(hide yes)
@@
 			(project "OpenAIO-Whoop"
 				(path "/2c3a7206-1e66-4d43-a02f-491225e20dd6/8d214749-72cf-5803-99b7-260f0c3f1838"
-					(reference "#PWR239")
+					(reference "#PWR226")
 					(unit 1)
 				)
@@
 		(in_pos_files no)
 		(dnp no)
-		(property "Reference" "#PWR245"
+		(property "Reference" "#PWR232"
 			(at 167.64 133.35 0)
 			(hide yes)
@@
 			(project "OpenAIO-Whoop"
 				(path "/2c3a7206-1e66-4d43-a02f-491225e20dd6/8d214749-72cf-5803-99b7-260f0c3f1838"
-					(reference "#PWR245")
+					(reference "#PWR232")
 					(unit 1)
 				)
@@
 		(in_pos_files no)
 		(dnp no)
-		(property "Reference" "#PWR246"
+		(property "Reference" "#PWR233"
 			(at 173.99 133.35 0)
 			(hide yes)
@@
 			(project "OpenAIO-Whoop"
 				(path "/2c3a7206-1e66-4d43-a02f-491225e20dd6/8d214749-72cf-5803-99b7-260f0c3f1838"
-					(reference "#PWR246")
+					(reference "#PWR233")
 					(unit 1)
 				)
@@
 		(in_pos_files no)
 		(dnp no)
-		(property "Reference" "#PWR247"
+		(property "Reference" "#PWR234"
 			(at 238.76 123.19 0)
 			(hide yes)
@@
 			)
 		)
-		(property "Value" "+5V_HD"
+		(property "Value" "+5V_BST"
 			(at 238.76 130.556 0)
 			(show_name no)
@@
 			(project "OpenAIO-Whoop"
 				(path "/2c3a7206-1e66-4d43-a02f-491225e20dd6/8d214749-72cf-5803-99b7-260f0c3f1838"
-					(reference "#PWR247")
+					(reference "#PWR234")
 					(unit 1)
 				)
@@
 		(in_pos_files no)
 		(dnp no)
-		(property "Reference" "#FLG08"
+		(property "Reference" "#FLG07"
 			(at 382.27 56.515 0)
 			(hide yes)
@@
 			(project "OpenAIO-Whoop"
 				(path "/2c3a7206-1e66-4d43-a02f-491225e20dd6/8d214749-72cf-5803-99b7-260f0c3f1838"
-					(reference "#FLG08")
+					(reference "#FLG07")
 					(unit 1)
 				)
@@
 		(in_pos_files no)
 		(dnp no)
-		(property "Reference" "#PWR244"
+		(property "Reference" "#PWR231"
 			(at 139.7 123.19 0)
 			(hide yes)
@@
 			(project "OpenAIO-Whoop"
 				(path "/2c3a7206-1e66-4d43-a02f-491225e20dd6/8d214749-72cf-5803-99b7-260f0c3f1838"
-					(reference "#PWR244")
+					(reference "#PWR231")
 					(unit 1)
 				)
@@
 		(in_pos_files no)
 		(dnp no)
-		(property "Reference" "#PWR240"
+		(property "Reference" "#PWR227"
 			(at 379.73 49.53 0)
 			(hide yes)
@@
 			(project "OpenAIO-Whoop"
 				(path "/2c3a7206-1e66-4d43-a02f-491225e20dd6/8d214749-72cf-5803-99b7-260f0c3f1838"
-					(reference "#PWR240")
+					(reference "#PWR227")
 					(unit 1)
 				)
@@
 		(in_pos_files no)
 		(dnp no)
-		(property "Reference" "#PWR238"
+		(property "Reference" "#PWR225"
 			(at 347.98 49.53 0)
 			(hide yes)
@@
 			(project "OpenAIO-Whoop"
 				(path "/2c3a7206-1e66-4d43-a02f-491225e20dd6/8d214749-72cf-5803-99b7-260f0c3f1838"
-					(reference "#PWR238")
+					(reference "#PWR225")
 					(unit 1)
 				)
@@
 		(in_pos_files no)
 		(dnp no)
-		(property "Reference" "#PWR243"
+		(property "Reference" "#PWR230"
 			(at 129.54 133.35 0)
 			(hide yes)
@@
 			(project "OpenAIO-Whoop"
 				(path "/2c3a7206-1e66-4d43-a02f-491225e20dd6/8d214749-72cf-5803-99b7-260f0c3f1838"
-					(reference "#PWR243")
+					(reference "#PWR230")
 					(unit 1)
 				)
@@
 		(in_pos_files no)
 		(dnp no)
-		(property "Reference" "#PWR242"
+		(property "Reference" "#PWR229"
 			(at 50.8 123.19 0)
 			(hide yes)
@@
 			(project "OpenAIO-Whoop"
 				(path "/2c3a7206-1e66-4d43-a02f-491225e20dd6/8d214749-72cf-5803-99b7-260f0c3f1838"
-					(reference "#PWR242")
+					(reference "#PWR229")
 					(unit 1)
 				)
@@
 		(in_pos_files no)
 		(dnp no)
-		(property "Reference" "#PWR248"
+		(property "Reference" "#PWR235"
 			(at 248.92 133.35 0)
 			(hide yes)
@@
 			(project "OpenAIO-Whoop"
 				(path "/2c3a7206-1e66-4d43-a02f-491225e20dd6/8d214749-72cf-5803-99b7-260f0c3f1838"
-					(reference "#PWR248")
+					(reference "#PWR235")
 					(unit 1)
 				)
@@
 		(in_pos_files no)
 		(dnp no)
-		(property "Reference" "#PWR249"
+		(property "Reference" "#PWR236"
 			(at 170.18 128.27 0)
 			(hide yes)
@@
 			(project "OpenAIO-Whoop"
 				(path "/2c3a7206-1e66-4d43-a02f-491225e20dd6/8d214749-72cf-5803-99b7-260f0c3f1838"
-					(reference "#PWR249")
-					(unit 1)
-				)
+					(reference "#PWR236")
+					(unit 1)
+				)

Commit message: 5 V input: two Schottky diodes replace the TPS2116 mux and the SGM40661 (D118)
D9 VBUS -> +5V and D10 +5V_BST -> +5V, MSKSEMI MS2A40LDF DFN1610-2
(LCSC C7380000, imported with import_part.py; land spec PASS). U3, R7,
R8, U24, C131 removed; C128 is +5V bulk; PWR_FLAG on +5V. Board synced.

Stale schematic notes rewritten (O4 switch block now "HD_EN PULL-DOWN",
TVS, INA186 input RC, PA NTC, R67, GPIO4 control, root power table).

ERC 0 errors; check_netlist 7 ok; sch_integrate --check clean;
setup_board --check up to date; board_spec 31/31; sync dry run 0 changes;
DRC unchanged.

Co-Authored-By: Claude Opus 5.5 <noreply@anthropic.com>
Changed lines of the file:
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@@
 		)
 	)
-	(text_box "HD pads for the DJI O4 Lite (D13, D16): VHD = +5V_HD (U5, on with HD_EN), TX1/RX1 = UART0 GPIO16/17 (silk per D89) for MSP DisplayPort; no SBUS pad.\nAnalog builds: TX1/RX1 are the only free UART (D89). 3.3 V logic only: a 5 V TX on RX1 would exceed the unpowered pad limit during the ramp. Copper only (DNP, A16)."
+	(text_box "HD pads for the DJI O4 Lite (D13, D16): VHD = +5V_BST (boost output, no load switch, D114), TX1/RX1 = UART0 GPIO16/17 (silk per D89) for MSP DisplayPort; no SBUS pad.\nAnalog builds: TX1/RX1 are the only free UART (D89). 3.3 V logic only: a 5 V TX on RX1 would exceed the unpowered pad limit during the ramp. Copper only (DNP, A16)."
 		(exclude_from_sim no)
 		(at 223.52 147.32 0)
@@
 		(in_pos_files no)
 		(dnp no)
-		(property "Reference" "#PWR228"
+		(property "Reference" "#PWR220"
 			(at 30.48 133.35 0)
 			(hide yes)
@@
 			(project "OpenAIO-Whoop"
 				(path "/2c3a7206-1e66-4d43-a02f-491225e20dd6/8d214749-72cf-5803-99b7-260f0c3f1838"
-					(reference "#PWR228")
+					(reference "#PWR220")
 					(unit 1)
 				)
@@
 		(in_pos_files no)
 		(dnp no)
-		(property "Reference" "#PWR226"
+		(property "Reference" "#PWR218"
 			(at 367.03 49.53 0)
 			(hide yes)
@@
 			(project "OpenAIO-Whoop"
 				(path "/2c3a7206-1e66-4d43-a02f-491225e20dd6/8d214749-72cf-5803-99b7-260f0c3f1838"
-					(reference "#PWR226")
+					(reference "#PWR218")
 					(unit 1)
 				)
@@
 		(in_pos_files no)
 		(dnp no)
-		(property "Reference" "#PWR232"
+		(property "Reference" "#PWR224"
 			(at 167.64 133.35 0)
 			(hide yes)
@@
 			(project "OpenAIO-Whoop"
 				(path "/2c3a7206-1e66-4d43-a02f-491225e20dd6/8d214749-72cf-5803-99b7-260f0c3f1838"
-					(reference "#PWR232")
+					(reference "#PWR224")
 					(unit 1)
 				)
@@
 		(in_pos_files no)
 		(dnp no)
-		(property "Reference" "#PWR233"
+		(property "Reference" "#PWR225"
 			(at 173.99 133.35 0)
 			(hide yes)
@@
 			(project "OpenAIO-Whoop"
 				(path "/2c3a7206-1e66-4d43-a02f-491225e20dd6/8d214749-72cf-5803-99b7-260f0c3f1838"
-					(reference "#PWR233")
+					(reference "#PWR225")
 					(unit 1)
 				)
@@
 		(in_pos_files no)
 		(dnp no)
-		(property "Reference" "#PWR234"
+		(property "Reference" "#PWR226"
 			(at 238.76 123.19 0)
 			(hide yes)
@@
 			(project "OpenAIO-Whoop"
 				(path "/2c3a7206-1e66-4d43-a02f-491225e20dd6/8d214749-72cf-5803-99b7-260f0c3f1838"
-					(reference "#PWR234")
+					(reference "#PWR226")
 					(unit 1)
 				)
@@
 		(in_pos_files no)
 		(dnp no)
-		(property "Reference" "#FLG07"
+		(property "Reference" "#FLG08"
 			(at 382.27 56.515 0)
 			(hide yes)
@@
 			(project "OpenAIO-Whoop"
 				(path "/2c3a7206-1e66-4d43-a02f-491225e20dd6/8d214749-72cf-5803-99b7-260f0c3f1838"
-					(reference "#FLG07")
+					(reference "#FLG08")
 					(unit 1)
 				)
@@
 		(in_pos_files no)
 		(dnp no)
-		(property "Reference" "#PWR231"
+		(property "Reference" "#PWR223"
 			(at 139.7 123.19 0)
 			(hide yes)
@@
 			(project "OpenAIO-Whoop"
 				(path "/2c3a7206-1e66-4d43-a02f-491225e20dd6/8d214749-72cf-5803-99b7-260f0c3f1838"
-					(reference "#PWR231")
+					(reference "#PWR223")
 					(unit 1)
 				)
@@
 		(in_pos_files no)
 		(dnp no)
-		(property "Reference" "#PWR227"
+		(property "Reference" "#PWR219"
 			(at 379.73 49.53 0)
 			(hide yes)
@@
 			(project "OpenAIO-Whoop"
 				(path "/2c3a7206-1e66-4d43-a02f-491225e20dd6/8d214749-72cf-5803-99b7-260f0c3f1838"
-					(reference "#PWR227")
+					(reference "#PWR219")
 					(unit 1)
 				)
@@
 		(in_pos_files no)
 		(dnp no)
-		(property "Reference" "#PWR225"
+		(property "Reference" "#PWR217"
 			(at 347.98 49.53 0)
 			(hide yes)
@@
 			(project "OpenAIO-Whoop"
 				(path "/2c3a7206-1e66-4d43-a02f-491225e20dd6/8d214749-72cf-5803-99b7-260f0c3f1838"
-					(reference "#PWR225")
+					(reference "#PWR217")
 					(unit 1)
 				)
@@
 		(in_pos_files no)
 		(dnp no)
-		(property "Reference" "#PWR230"
+		(property "Reference" "#PWR222"
 			(at 129.54 133.35 0)
 			(hide yes)
@@
 			(project "OpenAIO-Whoop"
 				(path "/2c3a7206-1e66-4d43-a02f-491225e20dd6/8d214749-72cf-5803-99b7-260f0c3f1838"
-					(reference "#PWR230")
+					(reference "#PWR222")
 					(unit 1)
 				)
@@
 		(in_pos_files no)
 		(dnp no)
-		(property "Reference" "#PWR229"
+		(property "Reference" "#PWR221"
 			(at 50.8 123.19 0)
 			(hide yes)
@@
 			(project "OpenAIO-Whoop"
 				(path "/2c3a7206-1e66-4d43-a02f-491225e20dd6/8d214749-72cf-5803-99b7-260f0c3f1838"
-					(reference "#PWR229")
+					(reference "#PWR221")
 					(unit 1)
 				)
@@
 		(in_pos_files no)
 		(dnp no)
-		(property "Reference" "#PWR235"
+		(property "Reference" "#PWR227"
 			(at 248.92 133.35 0)
 			(hide yes)
@@
 			(project "OpenAIO-Whoop"
 				(path "/2c3a7206-1e66-4d43-a02f-491225e20dd6/8d214749-72cf-5803-99b7-260f0c3f1838"
-					(reference "#PWR235")
+					(reference "#PWR227")
 					(unit 1)
 				)
@@
 		(in_pos_files no)
 		(dnp no)
-		(property "Reference" "#PWR236"
+		(property "Reference" "#PWR228"
 			(at 170.18 128.27 0)
 			(hide yes)
@@
 			(project "OpenAIO-Whoop"
 				(path "/2c3a7206-1e66-4d43-a02f-491225e20dd6/8d214749-72cf-5803-99b7-260f0c3f1838"
-					(reference "#PWR236")
+					(reference "#PWR228")
 					(unit 1)
 				)

Commit message: RTC6705 pin 40 / pin 17 filters per OpenOSD-X; O4 pads TX0/RX0 (D119)
R89 51R + C135 1u on LDD2V5 (pin 40), R90 3.3k + C136 1u on AVDD_6.5
(pin 17, symbol pin retyped passive), PWR_FLAG on U19_LDD2V5. O4 pad
values TX1/RX1 -> TX0/RX0 to match Betaflight's UART0. PINMAP gyro
alignment note for the back-side U11. Board not synced (layout open).

ERC 0 errors; check_netlist 7 ok.

Co-Authored-By: Claude Opus 5.5 <noreply@anthropic.com>
Parts:
- J28: value TX1 -> TX0
- J29: value RX1 -> RX0
Changed lines of the file:
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@@
 		(in_pos_files no)
 		(dnp no)
-		(property "Reference" "#PWR220"
+		(property "Reference" "#PWR223"
 			(at 30.48 133.35 0)
 			(hide yes)
@@
 			(project "OpenAIO-Whoop"
 				(path "/2c3a7206-1e66-4d43-a02f-491225e20dd6/8d214749-72cf-5803-99b7-260f0c3f1838"
-					(reference "#PWR220")
+					(reference "#PWR223")
 					(unit 1)
 				)
@@
 		(in_pos_files no)
 		(dnp no)
-		(property "Reference" "#PWR218"
+		(property "Reference" "#PWR221"
 			(at 367.03 49.53 0)
 			(hide yes)
@@
 			(project "OpenAIO-Whoop"
 				(path "/2c3a7206-1e66-4d43-a02f-491225e20dd6/8d214749-72cf-5803-99b7-260f0c3f1838"
-					(reference "#PWR218")
+					(reference "#PWR221")
 					(unit 1)
 				)
@@
 		(in_pos_files no)
 		(dnp no)
-		(property "Reference" "#PWR224"
+		(property "Reference" "#PWR227"
 			(at 167.64 133.35 0)
 			(hide yes)
@@
 			(project "OpenAIO-Whoop"
 				(path "/2c3a7206-1e66-4d43-a02f-491225e20dd6/8d214749-72cf-5803-99b7-260f0c3f1838"
-					(reference "#PWR224")
+					(reference "#PWR227")
 					(unit 1)
 				)
@@
 			)
 		)
-		(property "Value" "TX1"
+		(property "Value" "TX0"
 			(at 259.08 113.538 90)
 			(show_name no)
@@
 		(in_pos_files no)
 		(dnp no)
-		(property "Reference" "#PWR225"
+		(property "Reference" "#PWR228"
 			(at 173.99 133.35 0)
 			(hide yes)
@@
 			(project "OpenAIO-Whoop"
 				(path "/2c3a7206-1e66-4d43-a02f-491225e20dd6/8d214749-72cf-5803-99b7-260f0c3f1838"
-					(reference "#PWR225")
+					(reference "#PWR228")
 					(unit 1)
 				)
@@
 		(in_pos_files no)
 		(dnp no)
-		(property "Reference" "#PWR226"
+		(property "Reference" "#PWR229"
 			(at 238.76 123.19 0)
 			(hide yes)
@@
 			(project "OpenAIO-Whoop"
 				(path "/2c3a7206-1e66-4d43-a02f-491225e20dd6/8d214749-72cf-5803-99b7-260f0c3f1838"
-					(reference "#PWR226")
+					(reference "#PWR229")
 					(unit 1)
 				)
@@
 		(in_pos_files no)
 		(dnp no)
-		(property "Reference" "#FLG08"
+		(property "Reference" "#FLG09"
 			(at 382.27 56.515 0)
 			(hide yes)
@@
 			(project "OpenAIO-Whoop"
 				(path "/2c3a7206-1e66-4d43-a02f-491225e20dd6/8d214749-72cf-5803-99b7-260f0c3f1838"
-					(reference "#FLG08")
+					(reference "#FLG09")
 					(unit 1)
 				)
@@
 		(in_pos_files no)
 		(dnp no)
-		(property "Reference" "#PWR223"
+		(property "Reference" "#PWR226"
 			(at 139.7 123.19 0)
 			(hide yes)
@@
 			(project "OpenAIO-Whoop"
 				(path "/2c3a7206-1e66-4d43-a02f-491225e20dd6/8d214749-72cf-5803-99b7-260f0c3f1838"
-					(reference "#PWR223")
+					(reference "#PWR226")
 					(unit 1)
 				)
@@
 		(in_pos_files no)
 		(dnp no)
-		(property "Reference" "#PWR219"
+		(property "Reference" "#PWR222"
 			(at 379.73 49.53 0)
 			(hide yes)
@@
 			(project "OpenAIO-Whoop"
 				(path "/2c3a7206-1e66-4d43-a02f-491225e20dd6/8d214749-72cf-5803-99b7-260f0c3f1838"
-					(reference "#PWR219")
+					(reference "#PWR222")
 					(unit 1)
 				)
@@
 		(in_pos_files no)
 		(dnp no)
-		(property "Reference" "#PWR217"
+		(property "Reference" "#PWR220"
 			(at 347.98 49.53 0)
 			(hide yes)
@@
 			(project "OpenAIO-Whoop"
 				(path "/2c3a7206-1e66-4d43-a02f-491225e20dd6/8d214749-72cf-5803-99b7-260f0c3f1838"
-					(reference "#PWR217")
+					(reference "#PWR220")
 					(unit 1)
 				)
@@
 			)
 		)
-		(property "Value" "RX1"
+		(property "Value" "RX0"
 			(at 269.24 113.538 90)
 			(show_name no)
@@
 		(in_pos_files no)
 		(dnp no)
-		(property "Reference" "#PWR222"
+		(property "Reference" "#PWR225"
 			(at 129.54 133.35 0)
 			(hide yes)
@@
 			(project "OpenAIO-Whoop"
 				(path "/2c3a7206-1e66-4d43-a02f-491225e20dd6/8d214749-72cf-5803-99b7-260f0c3f1838"
-					(reference "#PWR222")
+					(reference "#PWR225")
 					(unit 1)
 				)
@@
 		(in_pos_files no)
 		(dnp no)
-		(property "Reference" "#PWR221"
+		(property "Reference" "#PWR224"
 			(at 50.8 123.19 0)
 			(hide yes)
@@
 			(project "OpenAIO-Whoop"
 				(path "/2c3a7206-1e66-4d43-a02f-491225e20dd6/8d214749-72cf-5803-99b7-260f0c3f1838"
-					(reference "#PWR221")
+					(reference "#PWR224")
 					(unit 1)
 				)
@@
 		(in_pos_files no)
 		(dnp no)
-		(property "Reference" "#PWR227"
+		(property "Reference" "#PWR230"
 			(at 248.92 133.35 0)
 			(hide yes)
@@
 			(project "OpenAIO-Whoop"
 				(path "/2c3a7206-1e66-4d43-a02f-491225e20dd6/8d214749-72cf-5803-99b7-260f0c3f1838"
-					(reference "#PWR227")
+					(reference "#PWR230")
 					(unit 1)
 				)
@@
 		(in_pos_files no)
 		(dnp no)
-		(property "Reference" "#PWR228"
+		(property "Reference" "#PWR231"
 			(at 170.18 128.27 0)
 			(hide yes)
@@
 			(project "OpenAIO-Whoop"
 				(path "/2c3a7206-1e66-4d43-a02f-491225e20dd6/8d214749-72cf-5803-99b7-260f0c3f1838"
-					(reference "#PWR228")
-					(unit 1)
-				)
+					(reference "#PWR231")
+					(unit 1)
+				)

Commit message: Footprint audit vs datasheets, 0201 lands to Murata minimum, schematic notes shortened
Footprints: 45 checked against their datasheets by group, no pin or
land errors. C/R/L_0201_..._L pad height 0.28 -> 0.30 (Murata GRM03
reflow table c >= 0.30); other lands already at least density per D109
and left unchanged. Land spec texts cleaned (sources, shared parts).

Schematic notes: 157 -> 152 items, 19.5k -> 9.7k characters, all
current (diode-OR, removed parts, RTC6705 filters, TX0/RX0).

check_footprint 107/107 lib specs PASS; ERC 0 errors / 2 warnings;
check_netlist 7 ok; sch_integrate --check clean. Board not synced.

Co-Authored-By: Claude Opus 5.5 <noreply@anthropic.com>
Other:
- note added: "MOTOR LANDS M1-M4"
- note removed: "Motor lands M1-M4: plug-ready, Molex PicoBlade header DNP"
Changed lines of the file:
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@@
 		)
 	)
-	(text "Motor lands M1-M4: plug-ready, Molex PicoBlade header DNP"
+	(text "MOTOR LANDS M1-M4"
 		(exclude_from_sim no)
 		(at 160.02 21.59 0)
@@
 		)
 	)
-	(text_box "Camera: JST SUR 0.8 mm plug J32 and pads CAM / GND / 5V in parallel (D63, D64), one mating zone (D72). VIDEO_IN -> OSD sheet (Analog class); +5V_CAM via FB1 on POWER, 0.12 A.\nGate G1 open: plug pin order provisional until a C03 lead is measured (a mirrored footprint puts 5 V on the camera's video output)."
+	(text_box "J32 JST SUR 0.8 mm plug and CAM / GND / 5V pads in parallel. VIDEO_IN (Analog class); +5V_CAM via FB1, 0.12 A.\nPlug pin order unverified: a mirrored plug puts 5 V on the video pin."
 		(exclude_from_sim no)
 		(at 104.14 147.32 0)
@@
 		)
 	)
-	(text_box "H1-H3: 25.5 mm M1.4 pattern (D73) cut in Edge.Cuts; symbols excluded from board, BOM and CPL, no net."
+	(text_box "H1-H3: 25.5 mm M1.4 pattern cut in Edge.Cuts; no net, not in BOM or CPL."
 		(exclude_from_sim no)
 		(at 17.78 203.2 0)
@@
 		)
 	)
-	(text_box "USB: J31 JST SH 4-pin vertical (D76; D72 side-entry withdrawn), BetaFPV order 1 GND, 2 D-, 3 D+, 4 VBUS. Pin 1 = GND is inferred: gate V0-USB before the P5 freeze (a mirrored plug puts -5 V on the OVP input).\nD7 TPD2EUSB30 ESD at J31, ahead of the 27R at the MCU. USB pair 90 Ohm, length-matched (D33). VBUS -> POWER (U24 OVP, D57); PWR_FLAG here."
+	(text_box "J31 JST SH 4-pin: 1 GND, 2 D-, 3 D+, 4 VBUS. Pin 1 = GND is unverified: check before freeze.\nD7 ESD at J31. USB pair 90 Ohm, length-matched. VBUS -> POWER."
 		(exclude_from_sim no)
 		(at 254 73.66 0)
@@
 		)
 	)
-	(text_box "HD pads for the DJI O4 Lite (D13, D16): VHD = +5V_BST (boost output, no load switch, D114), TX1/RX1 = UART0 GPIO16/17 (silk per D89) for MSP DisplayPort; no SBUS pad.\nAnalog builds: TX1/RX1 are the only free UART (D89). 3.3 V logic only: a 5 V TX on RX1 would exceed the unpowered pad limit during the ramp. Copper only (DNP, A16)."
+	(text_box "VHD = +5V_BST, TX0/RX0 = UART0 GPIO16/17 for MSP DisplayPort. 3.3 V logic only. Copper only (DNP)."
 		(exclude_from_sim no)
 		(at 223.52 147.32 0)
@@
 		)
 	)
-	(text_box "Row GND LED 5V BZ- (D63, D64; own GND pad J33 supersedes D27). LED = LED_STRIP straight from GPIO5, no translator (D52); a dead first LED is the level-problem symptom (V9). 5V feeds the strip and the buzzer, BZ- = drain of Q26 (RP2350A sheet). Copper only (DNP, A16)."
+	(text_box "Row GND LED 5V BZ-. LED = LED_STRIP straight from GPIO5 (3.3 V logic). 5V feeds strip and buzzer; BZ- = drain of Q26. Copper only (DNP)."
 		(exclude_from_sim no)
 		(at 17.78 147.32 0)
@@
 		)
 	)
-	(text_box "Battery pads J2 (+, CSA+) / J3 (-, GND) are drawn on the POWER sheet (D113): D1.7 mm plated pads (D101) for a user-fitted BT2.0 pigtail, >= 12 power vias each (D72). 1S only, 3.0-4.35 V (D14). Copper only (DNP, A16)."
+	(text_box "Battery pads J2 (+) / J3 (-) are drawn on POWER: 1.7 mm plated pads, >= 12 power vias each. 1S only, 3.0-4.35 V. Copper only (DNP)."
 		(exclude_from_sim no)
 		(at 17.78 25.4 0)
@@
 		)
 	)
-	(text_box "Motor lands (D65, Matrix 1S 5IN1 II style): one PicoBlade land per motor, pads 1/2/3 = PHASE_C/B/A; phase order is free, Bluejay sets the direction. On the top side, mouths facing out (D72).\nSolder the motor wires (default) or fit the DNP Molex 53047-0310 header: its 1.0 A contact rating is below the motor current, plugged motors run at the user's risk (README); V4 records the header temperature.\nM1 rear right, M2 front right, M3 rear left, M4 front left (Betaflight quad-X)."
+	(text_box "One PicoBlade land per motor, pads 1/2/3 = PHASE_C/B/A (order free, Bluejay sets direction). Top side, mouths facing out.\nSolder the wires or fit the DNP header 53047-0310 (1.0 A contact, below motor current)."
 		(exclude_from_sim no)
 		(at 76.2 53.34 0)
@@
 		)
 	)
-	(text_box "PADS: every off-board connection, style from the OpenFC-Lite(-Mini) pads sheets. Solder pads are DNP and out of BOM / CPL (LINEUP A16); the motor header is a DNP BOM line. 20 hierarchical labels = the sheet pins. TX1/RX1 = UART0, the only free UART (D89).\nOwed: J31 pin 1 = GND (V0-USB), J32 pin order (G1), motor-header temperature (V4)."
+	(text_box "PADS: every off-board connection. Solder pads are DNP and out of BOM / CPL.\nOpen: J31 pin 1 = GND, J32 pin order, motor-header temperature."
 		(exclude_from_sim no)
 		(at 101.6 182.88 0)
