File: hardware/pads.kicad_sch (KiCad schematic)
At the start: 21 parts, among them J10 M3, J13 M4, J20 LED, J21 5V, J22 BZ-, J23 CAM, J24 5V, J25 GND, J26 VHD, J27 GND, J28 TX0, J29 RX0, J31 USB, J32 CAM, J33 GND, J4 M1, J7 M2

Commit message: Larger solder pads and ESC programming pads, R1 shunt flipped (D120)
All hand-solder pads J20-J29/J33 on SolderPad_1.0x1.2mm; ESC C2 test
pads TP1-TP8 on TestPoint_Pad_D0.8mm; R1 rotated 270 without mirror
(owner edit, Kelvin pairs and INA186 polarity unchanged). ERC 0 errors;
check_netlist 7 ok.

Co-Authored-By: Claude Opus 5.5 <noreply@anthropic.com>
Parts:
- J20, J21, J22, J23, J24, J25, J26, J27, J28, J29, J33: footprint lib:SolderPad_0.8x1.0mm -> lib:SolderPad_1.0x1.2mm
Changed lines of the file:
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@@
 			)
 		)
-		(property "Footprint" "lib:SolderPad_0.8x1.0mm"
+		(property "Footprint" "lib:SolderPad_1.0x1.2mm"
 			(at 40.64 116.84 0)
 			(hide yes)
@@
 			)
 		)
-		(property "Footprint" "lib:SolderPad_0.8x1.0mm"
+		(property "Footprint" "lib:SolderPad_1.0x1.2mm"
 			(at 238.76 116.84 0)
 			(hide yes)
@@
 			)
 		)
-		(property "Footprint" "lib:SolderPad_0.8x1.0mm"
+		(property "Footprint" "lib:SolderPad_1.0x1.2mm"
 			(at 259.08 116.84 0)
 			(hide yes)
@@
 			)
 		)
-		(property "Footprint" "lib:SolderPad_0.8x1.0mm"
+		(property "Footprint" "lib:SolderPad_1.0x1.2mm"
 			(at 129.54 116.84 0)
 			(hide yes)
@@
 			)
 		)
-		(property "Footprint" "lib:SolderPad_0.8x1.0mm"
+		(property "Footprint" "lib:SolderPad_1.0x1.2mm"
 			(at 30.48 116.84 0)
 			(hide yes)
@@
 			)
 		)
-		(property "Footprint" "lib:SolderPad_0.8x1.0mm"
+		(property "Footprint" "lib:SolderPad_1.0x1.2mm"
 			(at 248.92 116.84 0)
 			(hide yes)
@@
 			)
 		)
-		(property "Footprint" "lib:SolderPad_0.8x1.0mm"
+		(property "Footprint" "lib:SolderPad_1.0x1.2mm"
 			(at 60.96 116.84 0)
 			(hide yes)
@@
 			)
 		)
-		(property "Footprint" "lib:SolderPad_0.8x1.0mm"
+		(property "Footprint" "lib:SolderPad_1.0x1.2mm"
 			(at 50.8 116.84 0)
 			(hide yes)
@@
 			)
 		)
-		(property "Footprint" "lib:SolderPad_0.8x1.0mm"
+		(property "Footprint" "lib:SolderPad_1.0x1.2mm"
 			(at 269.24 116.84 0)
 			(hide yes)
@@
 			)
 		)
-		(property "Footprint" "lib:SolderPad_0.8x1.0mm"
+		(property "Footprint" "lib:SolderPad_1.0x1.2mm"
 			(at 119.38 116.84 0)
 			(hide yes)
@@
 			)
 		)
-		(property "Footprint" "lib:SolderPad_0.8x1.0mm"
+		(property "Footprint" "lib:SolderPad_1.0x1.2mm"
 			(at 139.7 116.84 0)
 			(hide yes)
