File: hardware/imu.kicad_sch (KiCad schematic)
At the start: 5 parts, among them U11 BMI270, U12 TPS7A2018

Commit message: Correct Whoop schematic and prepare component library for routing
Add local BMI270 bypassing, improve regulator capacitance margin, isolate
bidirectional DShot supply domains, and correct PA reference accuracy.
Remove Q28/R11 with matching firmware polarity and retain the proven
OpenFC-Lite OSD topology. Correct the receiver LED bypass rail.

Synchronize PCB connectivity, verify component pins and land patterns,
and provide firmware bindings plus placement/layer guidance. Replace stale
manual BOM and interface plans with schematic-derived exports.

Validation: ERC 0, seven netlist checks, 48 footprint checks, 22 rule
behavior cases, and PCB schematic parity 0. The parked PCB retains layout
DRC findings and 499 unconnected items; no manufacturing or flight release.
Parts:
- added C137, C138: 100nF, lib:C_0201_0603Metric_L, symbol Device:C
- C61, C62: value 1uF -> 4.7uF; LCSC C76935 -> C335103; MPN GRM033R61A105ME44D -> GRM035R60J475ME15D
Connections:
- net +1.8V_GYRO: now also C138.1
- net +3.3V: now also C137.1
- net GND: now also C137.2, C138.2
