File: hardware/osd.kicad_sch (KiCad schematic)
At the start: 12 parts, among them U14 SN74LVC1G3157, U15 TLV7031

Commit message: Preserve owner schematic and placement edits before GPIO remap
Retain the saved layout, OSD bypass addition and component removals exactly
as received. This snapshot separates owner changes from the GPIO remap.
Parts:
- added C71: 100nF, lib:C_0201_0603Metric_L, symbol Device:C
Connections:
- net +3.3V: now also C71.1
- net GND: now also C71.2
