File: hardware/blackbox.kicad_sch (KiCad schematic)
At the start: 3 parts, among them U13 PY25Q128HA-DFH-IR

Commit message: Route USB and support links; correct flash mechanical tabs
Connections:
- no-connect marks 1 -> 0
Changed lines of the file:
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@@
 		)
 	)
-	(text_box "WP# and HOLD# tied to +3.3V for single-SPI operation; pin 7 must not float.\nR50 10k holds CS# high through reset. EP tabs no-connect."
+	(text_box "WP# and HOLD# tied to +3.3V for single-SPI operation; pin 7 must not float.\nR50 10k holds CS# high through reset. Unnumbered package tabs: floating mechanical lands."
 		(exclude_from_sim no)
 		(at 118.11 21.59 0)
@@
 		(diameter 0)
 		(color 0 0 0 0)
-	)
-	(no_connect
-		(at 77.47 78.74)
 	)
 	(wire
@@
 			)
 		)
-		(property "Description" "128 Mbit (16 MB) serial NOR flash, SPI/Dual/Quad/QPI, 2.7-3.6 V, -40..85 C, fC 133 MHz (READ 03h 80 MHz), USON-8 3x3x0.55 mm P0.8 (package DF), JEDEC ID 85 20 18 (Betaflight m25p16 table 'PUYA PY25Q128'); EP (9) = two exposed tie-bar tabs, no electrical role stated: leave unconnected with a no-connect flag"
+		(property "Description" "PY25Q128HA-DFH-IR, single-SPI mode; WP and HOLD are inputs. Quad mode is not supported by this symbol.; two unnumbered centre package tabs have no electrical terminal assignment in Puya Table 3-1/QRPD-0077; retain floating mechanical lands"
 			(at 76.2 68.58 0)
 			(hide yes)
@@
 		(pin "8"
 		)
-		(pin "9"
-		)
 		(instances
