File: hardware/OpenAIO-Whoop.kicad_sch (KiCad schematic)
At the start: 0 parts

Commit message: Owner: drop U24 level shifter, 1k series resistors on the motor lines (WIP save)
Co-Authored-By: Claude Opus 5.5 <noreply@anthropic.com>
Other:
- sheet RP2350A ports: added MOTOR1_FC, MOTOR2_FC, MOTOR3_FC, MOTOR4_FC; removed MOTOR1, MOTOR2, MOTOR3, MOTOR4
Changed lines of the file:
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@@
-			)
-		)
-		(pin "MOTOR1" bidirectional
-			(at 198.12 96.52 0)
-			(effects
-				(font
-					(size 1.27 1.27)
-				)
-				(justify right)
-			)
-		)
-		(pin "MOTOR2" bidirectional
-			(at 198.12 116.84 0)
-			(effects
-				(font
-					(size 1.27 1.27)
-				)
-				(justify right)
-			)
-		)
-		(pin "MOTOR3" bidirectional
-			(at 198.12 137.16 0)
-			(effects
-				(font
-					(size 1.27 1.27)
-				)
-				(justify right)
-			)
-		)
-		(pin "MOTOR4" bidirectional
-			(at 198.12 157.48 0)
-			(effects
-				(font
-					(size 1.27 1.27)
-				)
-				(justify right)
 			)
 		)
@@
 			(effects
 				(font
+					(size 1.27 1.27)
+				)
+				(justify right)
+			)
+		)
+		(pin "MOTOR1_FC" input
+			(at 198.12 96.52 0)
+			(effects
+				(font
+					(size 1.27 1.27)
+				)
+				(justify right)
+			)
+		)
+		(pin "MOTOR2_FC" input
+			(at 198.12 116.84 0)
+			(effects
+				(font
+					(size 1.27 1.27)
+				)
+				(justify right)
+			)
+		)
+		(pin "MOTOR3_FC" input
+			(at 198.12 137.16 0)
+			(effects
+				(font
+					(size 1.27 1.27)
+				)
+				(justify right)
+			)
+		)
+		(pin "MOTOR4_FC" input
+			(at 198.12 157.48 0)
+			(effects
+				(font
