File: hardware/esc_channel.kicad_sch (KiCad schematic)
At the start: 19 parts, among them Q29 AGM210MAP, Q30 AGM210MAP, Q31 AGM210MAP, U6 EFM8BB51F16I

Commit message: fix(schematic-review): BEMF check N7, review docs, D125 (#14)
* docs+check: BEMF phase-sense rule N7, review docs (limits, VTX path, Wi-Fi network absent, D125)

Schematic edits (BEMF swap, U4 text box, J2 note) are listed as manual Eeschema
steps in the PR: kicad-skip 0.2.5 does not round-trip these KiCad 10 files.

Co-Authored-By: Claude Opus 5.5 <noreply@anthropic.com>

* docs(readme): limits and VTX path tables under Constraints (keeps check_conventions D2 at base)

Co-Authored-By: Claude Opus 5.5 <noreply@anthropic.com>

* fix(sch): swap BEMF_B/BEMF_C labels in esc_channel (all four ESCs); correct U4 text box; 1S note at J2

Structured s-expression edit (sexpdata), re-saved by kicad-cli sch upgrade --force;
diff against the baseline re-save contains only the intended changes.

Co-Authored-By: Claude Opus 5.5 <noreply@anthropic.com>

---------

Co-authored-by: Claude Opus 5.5 <noreply@anthropic.com>
Parts:
- renumbered C22 to C24, C19 to C25, C20 to C26, C21 to C27, C23 to C29, C34 to C36, Q29 to Q32, Q30 to Q33, Q31 to Q34, R12 to R19, R13 to R20, R14 to R21, R15 to R22, R16 to R23, R17 to R24, R18 to R25, TP1 to TP3, TP2 to TP4, U6 to U7
Connections:
- net BEMF_B: now also R22.2; no longer R21.2
- net BEMF_C: now also R21.2; no longer R22.2
Changed lines of the file:
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@@
 		)
 	)
-	(label "BEMF_C"
+	(label "BEMF_B"
 		(at 165.1 63.5 0)
 		(effects
@@
 		)
 	)
-	(label "BEMF_B"
+	(label "BEMF_C"
 		(at 165.1 45.72 0)
 		(effects
@@
 		(in_pos_files no)
 		(dnp no)
-		(property "Reference" "#PWR42"
+		(property "Reference" "#PWR52"
 			(at 109.22 153.67 0)
 			(hide yes)
@@
 		(in_pos_files yes)
 		(dnp no)
-		(property "Reference" "R15"
+		(property "Reference" "R22"
 			(at 156.21 60.96 90)
 			(show_name no)
@@
 		(in_pos_files yes)
 		(dnp no)
-		(property "Reference" "U6"
+		(property "Reference" "U7"
 			(at 78.74 41.91 0)
 			(show_name no)
@@
 		(in_pos_files no)
 		(dnp no)
-		(property "Reference" "#PWR45"
+		(property "Reference" "#PWR55"
 			(at 99.06 177.8 0)
 			(hide yes)
@@
 		(in_pos_files yes)
 		(dnp no)
-		(property "Reference" "R16"
+		(property "Reference" "R23"
 			(at 156.21 33.02 90)
 			(show_name no)
@@
 		(in_pos_files yes)
 		(dnp no)
-		(property "Reference" "R13"
+		(property "Reference" "R20"
 			(at 156.21 25.4 90)
 			(show_name no)
@@
 		(in_pos_files yes)
 		(dnp no)
-		(property "Reference" "C19"
+		(property "Reference" "C25"
 			(at 60.96 35.56 0)
 			(show_name no)
@@
 		(in_pos_files yes)
 		(dnp no)
-		(property "Reference" "C34"
+		(property "Reference" "C36"
 			(at 80.645 142.24 0)
 			(show_name no)
@@
 		(in_pos_files yes)
 		(dnp no)
-		(property "Reference" "C20"
+		(property "Reference" "C26"
 			(at 68.58 142.24 0)
 			(show_name no)
@@
 		(in_pos_files yes)
 		(dnp no)
-		(property "Reference" "R12"
+		(property "Reference" "R19"
 			(at 40.64 63.5 90)
 			(show_name no)
@@
 		(in_pos_files yes)
 		(dnp no)
-		(property "Reference" "Q30"
+		(property "Reference" "Q33"
 			(at 101.6 152.4 0)
 			(show_name no)
@@
 		(in_pos_files no)
 		(dnp no)
-		(property "Reference" "#PWR46"
+		(property "Reference" "#PWR56"
 			(at 142.24 177.8 0)
 			(hide yes)
@@
 		(in_pos_files no)
 		(dnp no)
-		(property "Reference" "#PWR39"
+		(property "Reference" "#PWR49"
 			(at 76.2 87.63 0)
 			(hide yes)
@@
 		(in_pos_files yes)
 		(dnp no)
-		(property "Reference" "Q31"
+		(property "Reference" "Q34"
 			(at 144.78 152.4 0)
 			(show_name no)
@@
 		(in_pos_files no)
 		(dnp no)
-		(property "Reference" "#PWR0234"
+		(property "Reference" "#PWR0235"
 			(at 78.105 153.67 0)
 			(hide yes)
@@
 		(in_pos_files yes)
 		(dnp no)
-		(property "Reference" "R18"
+		(property "Reference" "R25"
 			(at 156.21 68.58 90)
 			(show_name no)
@@
 		(in_pos_files no)
 		(dnp no)
-		(property "Reference" "TP1"
+		(property "Reference" "TP3"
 			(at 110.49 64.77 90)
 			(show_name no)
@@
 		(in_pos_files no)
 		(dnp no)
-		(property "Reference" "TP2"
+		(property "Reference" "TP4"
 			(at 41.91 46.99 90)
 			(show_name no)
@@
 		(in_pos_files no)
 		(dnp no)
-		(property "Reference" "#PWR41"
+		(property "Reference" "#PWR51"
 			(at 66.04 153.67 0)
 			(hide yes)
@@
 		(in_pos_files yes)
 		(dnp no)
-		(property "Reference" "R17"
+		(property "Reference" "R24"
 			(at 156.21 50.8 90)
 			(show_name no)
@@
 		(in_pos_files yes)
 		(dnp no)
-		(property "Reference" "C21"
+		(property "Reference" "C27"
 			(at 154.94 142.24 0)
 			(show_name no)
@@
 		(in_pos_files no)
 		(dnp no)
-		(property "Reference" "#PWR37"
+		(property "Reference" "#PWR47"
 			(at 76.2 31.75 0)
 			(hide yes)
@@
 		(in_pos_files yes)
 		(dnp no)
-		(property "Reference" "C22"
+		(property "Reference" "C24"
 			(at 31.115 142.24 0)
 			(show_name no)
@@
 		(in_pos_files no)
 		(dnp no)
-		(property "Reference" "#PWR38"
+		(property "Reference" "#PWR48"
 			(at 58.42 49.53 0)
 			(hide yes)
@@
 		(in_pos_files no)
 		(dnp no)
-		(property "Reference" "#PWR0112"
+		(property "Reference" "#PWR0164"
 			(at 28.575 153.67 0)
 			(hide yes)
@@
 		(in_pos_files no)
 		(dnp no)
-		(property "Reference" "#PWR40"
+		(property "Reference" "#PWR50"
 			(at 22.86 143.51 0)
 			(hide yes)
@@
 		(in_pos_files yes)
 		(dnp no)
-		(property "Reference" "C23"
+		(property "Reference" "C29"
 			(at 111.76 142.24 0)
 			(show_name no)
@@
 		(in_pos_files no)
 		(dnp no)
-		(property "Reference" "#PWR44"
+		(property "Reference" "#PWR54"
 			(at 55.88 177.8 0)
 			(hide yes)
@@
 		(in_pos_files no)
 		(dnp no)
-		(property "Reference" "#PWR43"
+		(property "Reference" "#PWR53"
 			(at 152.4 153.67 0)
 			(hide yes)
@@
 		(in_pos_files yes)
 		(dnp no)
-		(property "Reference" "Q29"
+		(property "Reference" "Q32"
 			(at 58.42 152.4 0)
 			(show_name no)
@@
 		(in_pos_files yes)
 		(dnp no)
-		(property "Reference" "R14"
+		(property "Reference" "R21"
 			(at 156.21 43.18 90)
 			(show_name no)

Commit message: Owner: drop U24 level shifter, 1k series resistors on the motor lines (WIP save)
Co-Authored-By: Claude Opus 5.5 <noreply@anthropic.com>
Parts:
- removed R19: 22R, lib:R_0201_0603Metric_L, symbol Device:R
- renumbered C25 to C19, C26 to C20, C27 to C21, C24 to C22, C29 to C23, C36 to C34, Q32 to Q29, Q33 to Q30, Q34 to Q31, R20 to R13, R21 to R14, R22 to R15, R23 to R16, R24 to R17, R25 to R18, TP3 to TP1, TP4 to TP2, U7 to U6
Connections:
- net RTX is gone; now on net DSHOT: U6.17 (P0.5)
Changed lines of the file:
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@@
 	(wire
 		(pts
-			(xy 58.42 66.04) (xy 44.45 66.04)
-		)
-		(stroke
-			(width 0)
-			(type default)
-		)
-	)
-	(wire
-		(pts
 			(xy 149.86 35.56) (xy 152.4 35.56)
 		)
@@
 	(wire
 		(pts
-			(xy 36.83 66.04) (xy 31.75 66.04)
+			(xy 39.37 66.04) (xy 58.42 66.04)
 		)
 		(stroke
@@
 	(hierarchical_label "DSHOT"
 		(shape bidirectional)
-		(at 31.75 66.04 180)
+		(at 39.37 66.04 180)
 		(effects
 			(font
@@
 		(in_pos_files no)
 		(dnp no)
-		(property "Reference" "#PWR52"
+		(property "Reference" "#PWR42"
 			(at 109.22 153.67 0)
 			(hide yes)
@@
 		(in_pos_files yes)
 		(dnp no)
-		(property "Reference" "R22"
+		(property "Reference" "R15"
 			(at 156.21 60.96 90)
 			(show_name no)
@@
 		(in_pos_files yes)
 		(dnp no)
-		(property "Reference" "U7"
+		(property "Reference" "U6"
 			(at 78.74 41.91 0)
 			(show_name no)
@@
 		(in_pos_files no)
 		(dnp no)
-		(property "Reference" "#PWR55"
+		(property "Reference" "#PWR45"
 			(at 99.06 177.8 0)
 			(hide yes)
@@
 		(in_pos_files yes)
 		(dnp no)
-		(property "Reference" "R23"
+		(property "Reference" "R16"
 			(at 156.21 33.02 90)
 			(show_name no)
@@
 		(in_pos_files yes)
 		(dnp no)
-		(property "Reference" "R20"
+		(property "Reference" "R13"
 			(at 156.21 25.4 90)
 			(show_name no)
@@
 		(in_pos_files yes)
 		(dnp no)
-		(property "Reference" "C25"
+		(property "Reference" "C19"
 			(at 60.96 35.56 0)
 			(show_name no)
@@
 		(in_pos_files yes)
 		(dnp no)
-		(property "Reference" "C36"
+		(property "Reference" "C34"
 			(at 80.645 142.24 0)
 			(show_name no)
@@
 		(in_pos_files yes)
 		(dnp no)
-		(property "Reference" "C26"
+		(property "Reference" "C20"
 			(at 68.58 142.24 0)
 			(show_name no)
@@
 	)
 	(symbol
-		(lib_id "Device:R")
-		(at 40.64 66.04 90)
-		(unit 1)
-		(body_style 1)
-		(exclude_from_sim no)
-		(in_bom yes)
-		(on_board yes)
-		(in_pos_files yes)
-		(dnp no)
-		(property "Reference" "R19"
-			(at 40.64 63.5 90)
-			(show_name no)
-			(do_not_autoplace no)
-			(effects
-				(font
-					(size 1.27 1.27)
-				)
-			)
-		)
-		(property "Value" "22R"
-			(at 40.64 68.58 90)
-			(show_name no)
-			(do_not_autoplace no)
-			(effects
-				(font
-					(size 1.27 1.27)
-				)
-			)
-		)
-		(property "Footprint" "lib:R_0201_0603Metric_L"
-			(at 40.64 66.04 0)
-			(hide yes)
-			(show_name no)
-			(do_not_autoplace no)
-			(effects
-				(font
-					(size 1.27 1.27)
-				)
-			)
-		)
-		(property "Datasheet" "https://yageogroup.com/component-documentation/download/specsheet/RC0201FR-0722RL"
-			(at 40.64 66.04 0)
-			(hide yes)
-			(show_name no)
-			(do_not_autoplace no)
-			(effects
-				(font
-					(size 1.27 1.27)
-				)
-			)
-		)
-		(property "Description" "Resistor"
-			(at 40.64 66.04 0)
-			(hide yes)
-			(show_name no)
-			(do_not_autoplace no)
-			(effects
-				(font
-					(size 1.27 1.27)
-				)
-			)
-		)
-		(property "LCSC" "C155743"
-			(at 40.64 66.04 0)
-			(hide yes)
-			(show_name no)
-			(do_not_autoplace no)
-			(effects
-				(font
-					(size 1.27 1.27)
-				)
-			)
-		)
-		(property "MPN" "RC0201FR-0722RL"
-			(at 40.64 66.04 0)
-			(hide yes)
-			(show_name no)
-			(do_not_autoplace no)
-			(effects
-				(font
-					(size 1.27 1.27)
-				)
-			)
-		)
-		(property "Manufacturer" "Yageo"
-			(at 40.64 66.04 0)
-			(hide yes)
-			(show_name no)
-			(do_not_autoplace no)
-			(effects
-				(font
-					(size 1.27 1.27)
-				)
-			)
-		)
-		(pin "1"
-		)
-		(pin "2"
-		)
-		(instances
-			(project "OpenAIO-Whoop"
-				(path "/2c3a7206-1e66-4d43-a02f-491225e20dd6/0021bee0-9959-5c9e-86f0-21e49fa9ce8d"
-					(reference "R19")
-					(unit 1)
-				)
-				(path "/2c3a7206-1e66-4d43-a02f-491225e20dd6/6d139bfe-ad39-5d26-964c-e430887c2538"
-					(reference "R33")
-					(unit 1)
-				)
-				(path "/2c3a7206-1e66-4d43-a02f-491225e20dd6/a3c0517e-76c5-5fd7-8d0f-d7e948ad3995"
-					(reference "R26")
-					(unit 1)
-				)
-				(path "/2c3a7206-1e66-4d43-a02f-491225e20dd6/d67c44eb-67d1-5da8-b7a8-40b16f9433cd"
-					(reference "R12")
-					(unit 1)
-				)
-			)
-		)
-	)
-	(symbol
 		(lib_id "lib:AGM210MAP")
 		(at 96.52 158.75 0)
@@
 		(in_pos_files yes)
 		(dnp no)
-		(property "Reference" "Q33"
+		(property "Reference" "Q30"
 			(at 101.6 152.4 0)
 			(show_name no)
@@
 		(in_pos_files no)
 		(dnp no)
-		(property "Reference" "#PWR56"
+		(property "Reference" "#PWR46"
 			(at 142.24 177.8 0)
 			(hide yes)
@@
 		(in_pos_files no)
 		(dnp no)
-		(property "Reference" "#PWR49"
+		(property "Reference" "#PWR39"
 			(at 76.2 87.63 0)
 			(hide yes)
@@
 		(in_pos_files yes)
 		(dnp no)
-		(property "Reference" "Q34"
+		(property "Reference" "Q31"
 			(at 144.78 152.4 0)
 			(show_name no)
@@
 		(in_pos_files no)
 		(dnp no)
-		(property "Reference" "#PWR0235"
+		(property "Reference" "#PWR0234"
 			(at 78.105 153.67 0)
 			(hide yes)
@@
 		(in_pos_files yes)
 		(dnp no)
-		(property "Reference" "R25"
+		(property "Reference" "R18"
 			(at 156.21 68.58 90)
 			(show_name no)
@@
 		(in_pos_files no)
 		(dnp no)
-		(property "Reference" "TP3"
+		(property "Reference" "TP1"
 			(at 110.49 64.77 90)
 			(show_name no)
@@
 		(in_pos_files no)
 		(dnp no)
-		(property "Reference" "TP4"
+		(property "Reference" "TP2"
 			(at 41.91 46.99 90)
 			(show_name no)
@@
 		(in_pos_files no)
 		(dnp no)
-		(property "Reference" "#PWR51"
+		(property "Reference" "#PWR41"
 			(at 66.04 153.67 0)
 			(hide yes)
@@
 		(in_pos_files yes)
 		(dnp no)
-		(property "Reference" "R24"
+		(property "Reference" "R17"
 			(at 156.21 50.8 90)
 			(show_name no)
@@
 		(in_pos_files yes)
 		(dnp no)
-		(property "Reference" "C27"
+		(property "Reference" "C21"
 			(at 154.94 142.24 0)
 			(show_name no)
@@
 		(in_pos_files no)
 		(dnp no)
-		(property "Reference" "#PWR47"
+		(property "Reference" "#PWR37"
 			(at 76.2 31.75 0)
 			(hide yes)
@@
 		(in_pos_files yes)
 		(dnp no)
-		(property "Reference" "C24"
+		(property "Reference" "C22"
 			(at 31.115 142.24 0)
 			(show_name no)
@@
 		(in_pos_files no)
 		(dnp no)
-		(property "Reference" "#PWR48"
+		(property "Reference" "#PWR38"
 			(at 58.42 49.53 0)
 			(hide yes)
@@
 		(in_pos_files no)
 		(dnp no)
-		(property "Reference" "#PWR0164"
+		(property "Reference" "#PWR0112"
 			(at 28.575 153.67 0)
 			(hide yes)
@@
 		(in_pos_files no)
 		(dnp no)
-		(property "Reference" "#PWR50"
+		(property "Reference" "#PWR40"
 			(at 22.86 143.51 0)
 			(hide yes)
@@
 		(in_pos_files yes)
 		(dnp no)
-		(property "Reference" "C29"
+		(property "Reference" "C23"
 			(at 111.76 142.24 0)
 			(show_name no)
@@
 		(in_pos_files no)
 		(dnp no)
-		(property "Reference" "#PWR54"
+		(property "Reference" "#PWR44"
 			(at 55.88 177.8 0)
 			(hide yes)
@@
 		(in_pos_files no)
 		(dnp no)
-		(property "Reference" "#PWR53"
+		(property "Reference" "#PWR43"
 			(at 152.4 153.67 0)
 			(hide yes)
@@
 		(in_pos_files yes)
 		(dnp no)
-		(property "Reference" "Q32"
+		(property "Reference" "Q29"
 			(at 58.42 152.4 0)
 			(show_name no)
@@
 		(in_pos_files yes)
 		(dnp no)
-		(property "Reference" "R21"
+		(property "Reference" "R14"
 			(at 156.21 43.18 90)
 			(show_name no)

Commit message: Owner routing, per-ESC 22uF bulk caps, J34 removed (WIP save, unreviewed)
Co-Authored-By: Claude Opus 5.5 <noreply@anthropic.com>
Parts:
- added C53: 22uF, lib:C_0603_1608Metric_L, symbol Device:C
Connections:
- net +BATT: now also C53.1
- net GND: now also C53.2
Changed lines of the file:
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@@
 	)
 	(junction
+		(at 118.745 139.7)
+		(diameter 0)
+		(color 0 0 0 0)
+	)
+	(junction
 		(at 66.04 139.7)
 		(diameter 0)
@@
 	)
 	(symbol
+		(lib_id "power:GND")
+		(at 118.745 147.32 0)
+		(unit 1)
+		(body_style 1)
+		(exclude_from_sim no)
+		(in_bom no)
+		(on_board yes)
+		(in_pos_files no)
+		(dnp no)
+		(property "Reference" "#PWR0238"
+			(at 118.745 153.67 0)
+			(hide yes)
+			(show_name no)
+			(do_not_autoplace no)
+			(effects
+				(font
+					(size 1.27 1.27)
+				)
+			)
+		)
+		(property "Value" "GND"
+			(at 118.745 151.13 0)
+			(show_name no)
+			(do_not_autoplace no)
+			(effects
+				(font
+					(size 1.27 1.27)
+				)
+			)
+		)
+		(property "Footprint" ""
+			(at 118.745 147.32 0)
+			(hide yes)
+			(show_name no)
+			(do_not_autoplace no)
+			(effects
+				(font
+					(size 1.27 1.27)
+				)
+			)
+		)
+		(property "Datasheet" ""
+			(at 118.745 147.32 0)
+			(hide yes)
+			(show_name no)
+			(do_not_autoplace no)
+			(effects
+				(font
+					(size 1.27 1.27)
+				)
+			)
+		)
+		(property "Description" "Power symbol creates a global label with name \"GND\" , ground"
+			(at 118.745 147.32 0)
+			(hide yes)
+			(show_name no)
+			(do_not_autoplace no)
+			(effects
+				(font
+					(size 1.27 1.27)
+				)
+			)
+		)
+		(pin "1"
+		)
+		(instances
+			(project "OpenAIO-Whoop"
+				(path "/2c3a7206-1e66-4d43-a02f-491225e20dd6/0021bee0-9959-5c9e-86f0-21e49fa9ce8d"
+					(reference "#PWR0239")
+					(unit 1)
+				)
+				(path "/2c3a7206-1e66-4d43-a02f-491225e20dd6/6d139bfe-ad39-5d26-964c-e430887c2538"
+					(reference "#PWR0241")
+					(unit 1)
+				)
+				(path "/2c3a7206-1e66-4d43-a02f-491225e20dd6/a3c0517e-76c5-5fd7-8d0f-d7e948ad3995"
+					(reference "#PWR0240")
+					(unit 1)
+				)
+				(path "/2c3a7206-1e66-4d43-a02f-491225e20dd6/d67c44eb-67d1-5da8-b7a8-40b16f9433cd"
+					(reference "#PWR0238")
+					(unit 1)
+				)
+			)
+		)
+	)
+	(symbol
 		(lib_id "Device:R")
 		(at 156.21 35.56 90)
@@
 					(unit 1)
 				)
+			)
+		)
+	)
+	(symbol
+		(lib_id "Device:C")
+		(at 118.745 143.51 0)
+		(unit 1)
+		(body_style 1)
+		(exclude_from_sim no)
+		(in_bom yes)
+		(on_board yes)
+		(in_pos_files yes)
+		(dnp no)
+		(property "Reference" "C53"
+			(at 121.285 142.24 0)
+			(show_name no)
+			(do_not_autoplace no)
+			(effects
+				(font
+					(size 1.27 1.27)
+				)
+				(justify left)
+			)
+		)
+		(property "Value" "22uF"
+			(at 121.285 144.78 0)
+			(show_name no)
+			(do_not_autoplace no)
+			(effects
+				(font
+					(size 1.27 1.27)
+				)
+				(justify left)
+			)
+		)
+		(property "Footprint" "lib:C_0603_1608Metric_L"
+			(at 118.745 143.51 0)
+			(hide yes)
+			(show_name no)
+			(do_not_autoplace no)
+			(effects
+				(font
+					(size 1.27 1.27)
+				)
+			)
+		)
+		(property "Datasheet" ""
+			(at 118.745 143.51 0)
+			(hide yes)
+			(show_name no)
+			(do_not_autoplace no)
+			(effects
+				(font
+					(size 1.27 1.27)
+				)
+			)
+		)
+		(property "Description" "Unpolarized capacitor"
+			(at 118.745 143.51 0)
+			(hide yes)
+			(show_name no)
+			(do_not_autoplace no)
+			(effects
+				(font
+					(size 1.27 1.27)
+				)
+			)
+		)
+		(property "LCSC" "C393031"
+			(at 118.745 143.51 0)
+			(hide yes)
+			(show_name no)
+			(do_not_autoplace no)
+			(effects
+				(font
+					(size 1.27 1.27)
+				)
+			)
+		)
+		(property "MPN" "GRM188C80J226ME15D"
+			(at 118.745 143.51 0)
+			(hide yes)
+			(show_name no)
+			(do_not_autoplace no)
+			(effects
+				(font
+					(size 1.27 1.27)
+				)
+			)
+		)
+		(property "Manufacturer" "Murata"
+			(at 118.745 143.51 0)
+			(hide yes)
+			(show_name no)
+			(do_not_autoplace no)
+			(effects
+				(font
+					(size 1.27 1.27)
+				)
+			)
+		)
+		(pin "1"
+		)
+		(pin "2"
+		)
+		(instances
+			(project "OpenAIO-Whoop"
+				(path "/2c3a7206-1e66-4d43-a02f-491225e20dd6/0021bee0-9959-5c9e-86f0-21e49fa9ce8d"
+					(reference "C55")
+					(unit 1)
+				)
+				(path "/2c3a7206-1e66-4d43-a02f-491225e20dd6/6d139bfe-ad39-5d26-964c-e430887c2538"
+					(reference "C64")
+					(unit 1)
+				)
+				(path "/2c3a7206-1e66-4d43-a02f-491225e20dd6/a3c0517e-76c5-5fd7-8d0f-d7e948ad3995"
+					(reference "C63")
+					(unit 1)
+				)
+				(path "/2c3a7206-1e66-4d43-a02f-491225e20dd6/d67c44eb-67d1-5da8-b7a8-40b16f9433cd"
+					(reference "C53")
+					(unit 1)
+				)
