File: hardware/esc_channel.kicad_sch (KiCad schematic)
At the start: 19 parts, among them Q29 AGM210MAP, Q30 AGM210MAP, Q31 AGM210MAP, U6 EFM8BB51F16I

Commit message: Every schematic symbol project-local (Device, power, Connector, Mechanical moved into lib)
tools/localise_symbols.py from OpenAIO. Netlist identical, ERC unchanged (0 errors, 24 warnings), every symbol, footprint and 3D model resolves inside the repo.

Co-Authored-By: Claude Opus 5.5 <noreply@anthropic.com>
Parts:
- C24: renamed from C22; symbol Device:C -> lib:C
- C25: renamed from C19; symbol Device:C -> lib:C
- C26: renamed from C20; symbol Device:C -> lib:C
- C27: renamed from C21; symbol Device:C -> lib:C
- C29: renamed from C23; symbol Device:C -> lib:C
- C36: renamed from C34; symbol Device:C -> lib:C
- C55: renamed from C53; symbol Device:C -> lib:C
- R20: renamed from R13; symbol Device:R -> lib:R
- R21: renamed from R14; symbol Device:R -> lib:R
- R22: renamed from R15; symbol Device:R -> lib:R
- R23: renamed from R16; symbol Device:R -> lib:R
- R24: renamed from R17; symbol Device:R -> lib:R
- R25: renamed from R18; symbol Device:R -> lib:R
- TP3: renamed from TP1; symbol Connector:TestPoint -> lib:TestPoint
- TP4: renamed from TP2; symbol Connector:TestPoint -> lib:TestPoint
- renumbered Q29 to Q32, Q30 to Q33, Q31 to Q34, U6 to U7
Changed lines of the file:
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@@
 	)
 	(symbol
-		(lib_id "power:GND")
+		(lib_id "lib:GND")
 		(at 109.22 147.32 0)
 		(unit 1)
@@
 		(in_pos_files no)
 		(dnp no)
-		(property "Reference" "#PWR42"
+		(property "Reference" "#PWR52"
 			(at 109.22 153.67 0)
 			(hide yes)
@@
 	)
 	(symbol
-		(lib_id "Device:R")
+		(lib_id "lib:R")
 		(at 156.21 63.5 90)
 		(unit 1)
@@
 		(in_pos_files yes)
 		(dnp no)
-		(property "Reference" "R15"
+		(property "Reference" "R22"
 			(at 156.21 60.96 90)
 			(show_name no)
@@
 		(in_pos_files yes)
 		(dnp no)
-		(property "Reference" "U6"
+		(property "Reference" "U7"
 			(at 78.74 41.91 0)
 			(show_name no)
@@
 	)
 	(symbol
-		(lib_id "power:GND")
+		(lib_id "lib:GND")
 		(at 99.06 171.45 0)
 		(unit 1)
@@
 		(in_pos_files no)
 		(dnp no)
-		(property "Reference" "#PWR45"
+		(property "Reference" "#PWR55"
 			(at 99.06 177.8 0)
 			(hide yes)
@@
 	)
 	(symbol
-		(lib_id "power:GND")
+		(lib_id "lib:GND")
 		(at 118.745 147.32 0)
 		(unit 1)
@@
 		(in_pos_files no)
 		(dnp no)
-		(property "Reference" "#PWR0238"
+		(property "Reference" "#PWR0239"
 			(at 118.745 153.67 0)
 			(hide yes)
@@
 	)
 	(symbol
-		(lib_id "Device:R")
+		(lib_id "lib:R")
 		(at 156.21 35.56 90)
 		(unit 1)
@@
 		(in_pos_files yes)
 		(dnp no)
-		(property "Reference" "R16"
+		(property "Reference" "R23"
 			(at 156.21 33.02 90)
 			(show_name no)
@@
 	)
 	(symbol
-		(lib_id "Device:R")
+		(lib_id "lib:R")
 		(at 156.21 27.94 90)
 		(unit 1)
@@
 		(in_pos_files yes)
 		(dnp no)
-		(property "Reference" "R13"
+		(property "Reference" "R20"
 			(at 156.21 25.4 90)
 			(show_name no)
@@
 	)
 	(symbol
-		(lib_id "Device:C")
+		(lib_id "lib:C")
 		(at 58.42 36.83 0)
 		(unit 1)
@@
 		(in_pos_files yes)
 		(dnp no)
-		(property "Reference" "C19"
+		(property "Reference" "C25"
 			(at 60.96 35.56 0)
 			(show_name no)
@@
 	)
 	(symbol
-		(lib_id "Device:C")
+		(lib_id "lib:C")
 		(at 78.105 143.51 0)
 		(unit 1)
@@
 		(in_pos_files yes)
 		(dnp no)
-		(property "Reference" "C34"
+		(property "Reference" "C36"
 			(at 80.645 142.24 0)
 			(show_name no)
@@
 	)
 	(symbol
-		(lib_id "Device:C")
+		(lib_id "lib:C")
 		(at 66.04 143.51 0)
 		(unit 1)
@@
 		(in_pos_files yes)
 		(dnp no)
-		(property "Reference" "C20"
+		(property "Reference" "C26"
 			(at 68.58 142.24 0)
 			(show_name no)
@@
 		(in_pos_files yes)
 		(dnp no)
-		(property "Reference" "Q30"
+		(property "Reference" "Q33"
 			(at 101.6 152.4 0)
 			(show_name no)
@@
 	)
 	(symbol
-		(lib_id "power:GND")
+		(lib_id "lib:GND")
 		(at 142.24 171.45 0)
 		(unit 1)
@@
 		(in_pos_files no)
 		(dnp no)
-		(property "Reference" "#PWR46"
+		(property "Reference" "#PWR56"
 			(at 142.24 177.8 0)
 			(hide yes)
@@
 	)
 	(symbol
-		(lib_id "power:GND")
+		(lib_id "lib:GND")
 		(at 76.2 81.28 0)
 		(unit 1)
@@
 		(in_pos_files no)
 		(dnp no)
-		(property "Reference" "#PWR39"
+		(property "Reference" "#PWR49"
 			(at 76.2 87.63 0)
 			(hide yes)
@@
 		(in_pos_files yes)
 		(dnp no)
-		(property "Reference" "Q31"
+		(property "Reference" "Q34"
 			(at 144.78 152.4 0)
 			(show_name no)
@@
 	)
 	(symbol
-		(lib_id "power:GND")
+		(lib_id "lib:GND")
 		(at 78.105 147.32 0)
 		(unit 1)
@@
 		(in_pos_files no)
 		(dnp no)
-		(property "Reference" "#PWR0234"
+		(property "Reference" "#PWR0235"
 			(at 78.105 153.67 0)
 			(hide yes)
@@
 	)
 	(symbol
-		(lib_id "Device:R")
+		(lib_id "lib:R")
 		(at 156.21 71.12 90)
 		(unit 1)
@@
 		(in_pos_files yes)
 		(dnp no)
-		(property "Reference" "R18"
+		(property "Reference" "R25"
 			(at 156.21 68.58 90)
 			(show_name no)
@@
 	)
 	(symbol
-		(lib_id "Connector:TestPoint")
+		(lib_id "lib:TestPoint")
 		(at 106.68 68.58 270)
 		(unit 1)
@@
 		(in_pos_files no)
 		(dnp no)
-		(property "Reference" "TP1"
+		(property "Reference" "TP3"
 			(at 110.49 64.77 90)
 			(show_name no)
@@
 	)
 	(symbol
-		(lib_id "Connector:TestPoint")
+		(lib_id "lib:TestPoint")
 		(at 45.72 50.8 90)
 		(unit 1)
@@
 		(in_pos_files no)
 		(dnp no)
-		(property "Reference" "TP2"
+		(property "Reference" "TP4"
 			(at 41.91 46.99 90)
 			(show_name no)
@@
 	)
 	(symbol
-		(lib_id "power:GND")
+		(lib_id "lib:GND")
 		(at 66.04 147.32 0)
 		(unit 1)
@@
 		(in_pos_files no)
 		(dnp no)
-		(property "Reference" "#PWR41"
+		(property "Reference" "#PWR51"
 			(at 66.04 153.67 0)
 			(hide yes)
@@
 	)
 	(symbol
-		(lib_id "Device:R")
+		(lib_id "lib:R")
 		(at 156.21 53.34 90)
 		(unit 1)
@@
 		(in_pos_files yes)
 		(dnp no)
-		(property "Reference" "R17"
+		(property "Reference" "R24"
 			(at 156.21 50.8 90)
 			(show_name no)
@@
 	)
 	(symbol
-		(lib_id "Device:C")
+		(lib_id "lib:C")
 		(at 152.4 143.51 0)
 		(unit 1)
@@
 		(in_pos_files yes)
 		(dnp no)
-		(property "Reference" "C21"
+		(property "Reference" "C27"
 			(at 154.94 142.24 0)
 			(show_name no)
@@
 	)
 	(symbol
-		(lib_id "power:+BATT")
+		(lib_id "lib:+BATT")
 		(at 76.2 27.94 0)
 		(unit 1)
@@
 		(in_pos_files no)
 		(dnp no)
-		(property "Reference" "#PWR37"
+		(property "Reference" "#PWR47"
 			(at 76.2 31.75 0)
 			(hide yes)
@@
 	)
 	(symbol
-		(lib_id "Device:C")
+		(lib_id "lib:C")
 		(at 118.745 143.51 0)
 		(unit 1)
@@
 		(in_pos_files yes)
 		(dnp no)
-		(property "Reference" "C53"
+		(property "Reference" "C55"
 			(at 121.285 142.24 0)
 			(show_name no)
@@
 	)
 	(symbol
-		(lib_id "Device:C")
+		(lib_id "lib:C")
 		(at 28.575 143.51 0)
 		(unit 1)
@@
 		(in_pos_files yes)
 		(dnp no)
-		(property "Reference" "C22"
+		(property "Reference" "C24"
 			(at 31.115 142.24 0)
 			(show_name no)
@@
 	)
 	(symbol
-		(lib_id "power:GND")
+		(lib_id "lib:GND")
 		(at 58.42 43.18 0)
 		(unit 1)
@@
 		(in_pos_files no)
 		(dnp no)
-		(property "Reference" "#PWR38"
+		(property "Reference" "#PWR48"
 			(at 58.42 49.53 0)
 			(hide yes)
@@
 	)
 	(symbol
-		(lib_id "power:GND")
+		(lib_id "lib:GND")
 		(at 28.575 147.32 0)
 		(unit 1)
@@
 		(in_pos_files no)
 		(dnp no)
-		(property "Reference" "#PWR0112"
+		(property "Reference" "#PWR0164"
 			(at 28.575 153.67 0)
 			(hide yes)
@@
 	)
 	(symbol
-		(lib_id "power:+BATT")
+		(lib_id "lib:+BATT")
 		(at 22.86 139.7 0)
 		(unit 1)
@@
 		(in_pos_files no)
 		(dnp no)
-		(property "Reference" "#PWR40"
+		(property "Reference" "#PWR50"
 			(at 22.86 143.51 0)
 			(hide yes)
@@
 	)
 	(symbol
-		(lib_id "Device:C")
+		(lib_id "lib:C")
 		(at 109.22 143.51 0)
 		(unit 1)
@@
 		(in_pos_files yes)
 		(dnp no)
-		(property "Reference" "C23"
+		(property "Reference" "C29"
 			(at 111.76 142.24 0)
 			(show_name no)
@@
 	)
 	(symbol
-		(lib_id "power:GND")
+		(lib_id "lib:GND")
 		(at 55.88 171.45 0)
 		(unit 1)
@@
 		(in_pos_files no)
 		(dnp no)
-		(property "Reference" "#PWR44"
+		(property "Reference" "#PWR54"
 			(at 55.88 177.8 0)
 			(hide yes)
@@
 	)
 	(symbol
-		(lib_id "power:GND")
+		(lib_id "lib:GND")
 		(at 152.4 147.32 0)
 		(unit 1)
@@
 		(in_pos_files no)
 		(dnp no)
-		(property "Reference" "#PWR43"
+		(property "Reference" "#PWR53"
 			(at 152.4 153.67 0)
 			(hide yes)
@@
 		(in_pos_files yes)
 		(dnp no)
-		(property "Reference" "Q29"
+		(property "Reference" "Q32"
 			(at 58.42 152.4 0)
 			(show_name no)
@@
 	)
 	(symbol
-		(lib_id "Device:R")
+		(lib_id "lib:R")
 		(at 156.21 45.72 90)
 		(unit 1)
@@
 		(in_pos_files yes)
 		(dnp no)
-		(property "Reference" "R14"
+		(property "Reference" "R21"
 			(at 156.21 43.18 90)
 			(show_name no)
